File: LV_power.sch (KiCad schematic (older format))
At the start: 0 parts

Commit message: V0 schematic complete (?)
Parts:
- added C?: 10uF 50V, symbol C_Small
- added C?: 22uF 16V, symbol C_Small
- added C?: 100uF 16V, symbol C_Small
- added C?: 470nF, symbol C_Small
- added C? (x2): 10uF, symbol C_Small
- added CON?: BARREL_JACK, symbol BARREL_JACK
- added R?: 0R, symbol R_Small
- added U?: APE8865N-33-HF-3, SOT-23, symbol APE8865N-33-HF-3
- added U?: V7805-500-SMT, symbol V78-500-SMT
Connections:
- new net: C?.1, U?.6 (Vadj)
- new net +15V: C?.1, CON?.1, U?.1 (Vin)
- new net +3V3: C?.1, U?.2 (VOUT)
- new net +5VA: R?.2
- new net +5VD: C?.1, C?.1, C?.1, R?.1, U?.3 (VIN), U?.5 (Vout)
- new net GNDD: C?.2, C?.2, C?.2, C?.2, C?.2, C?.2, CON?.2, CON?.3, U?.1 (GND), U?.7 (GND), U?.9 (GND)

Commit message: Annotate, fix schematic DRC, footprint for DIMM100
Parts:
- R2: renamed from R?; value 0R -> 0R/BEAD
- gave numbers to parts that had none: 9
Connections:
- no-connect marks 0 -> 1
Changed lines of the file:
@@
 $EndDescr
 $Comp
-L BARREL_JACK CON?
+L BARREL_JACK CON1
 U 1 1 57A588D1
 P 2600 3550
-F 0 "CON?" H 2581 3875 50  0000 C CNN
+F 0 "CON1" H 2581 3875 50  0000 C CNN
 F 1 "BARREL_JACK" H 2581 3784 50  0000 C CNN
 F 2 "" H 2600 3550 50  0000 C CNN
@@
 $EndComp
 $Comp
-L APE8865N-33-HF-3 U?
+L APE8865N-33-HF-3 U2
 U 1 1 57A624B4
 P 7350 4150
-F 0 "U?" H 7350 4558 50  0000 C CNN
+F 0 "U2" H 7350 4558 50  0000 C CNN
 F 1 "APE8865N-33-HF-3" H 7350 4467 50  0000 C CNN
 F 2 "SOT-23" H 7350 4376 50  0000 C CIN
@@
 $EndComp
 $Comp
-L V78-500-SMT U?
+L V78-500-SMT U1
 U 1 1 57A628BE
 P 4700 3400
-F 0 "U?" H 4700 3687 60  0000 C CNN
+F 0 "U1" H 4700 3687 60  0000 C CNN
 F 1 "V7805-500-SMT" H 4700 3581 60  0000 C CNN
 F 2 "" H 4700 3400 60  0001 C CNN
@@
 $EndComp
 $Comp
-L +15V #PWR?
+L +15V #PWR018
 U 1 1 57A629B3
 P 3350 3350
-F 0 "#PWR?" H 3350 3200 50  0001 C CNN
+F 0 "#PWR018" H 3350 3200 50  0001 C CNN
 F 1 "+15V" H 3365 3523 50  0000 C CNN
 F 2 "" H 3350 3350 50  0000 C CNN
@@
 	2900 3550 2900 3650
 $Comp
-L GNDD #PWR?
+L GNDD #PWR019
 U 1 1 57A62A2D
 P 4500 3850
-F 0 "#PWR?" H 4500 3600 50  0001 C CNN
+F 0 "#PWR019" H 4500 3600 50  0001 C CNN
 F 1 "GNDD" H 4505 3677 50  0000 C CNN
 F 2 "" H 4500 3850 50  0000 C CNN
@@
 Connection ~ 3350 3450
 $Comp
-L C_Small C?
+L C_Small C1
 U 1 1 57A62AD5
 P 3600 3600
-F 0 "C?" H 3692 3646 50  0000 L CNN
+F 0 "C1" H 3692 3646 50  0000 L CNN
 F 1 "10uF 50V" H 3692 3555 50  0000 L CNN
 F 2 "" H 3600 3600 50  0000 C CNN
@@
 $EndComp
 $Comp
-L GNDD #PWR?
+L GNDD #PWR020
 U 1 1 57A62B8A
 P 3600 3750
-F 0 "#PWR?" H 3600 3500 50  0001 C CNN
+F 0 "#PWR020" H 3600 3500 50  0001 C CNN
 F 1 "GNDD" H 3605 3577 50  0000 C CNN
 F 2 "" H 3600 3750 50  0000 C CNN
@@
 Connection ~ 3600 3450
 $Comp
-L C_Small C?
+L C_Small C3
 U 1 1 57A62C61
 P 5350 3600
-F 0 "C?" H 5442 3646 50  0000 L CNN
+F 0 "C3" H 5442 3646 50  0000 L CNN
 F 1 "22uF 16V" H 5442 3555 50  0000 L CNN
 F 2 "" H 5350 3600 50  0000 C CNN
@@
 $EndComp
 $Comp
-L GNDD #PWR?
+L GNDD #PWR021
 U 1 1 57A62C67
 P 5350 3750
-F 0 "#PWR?" H 5350 3500 50  0001 C CNN
+F 0 "#PWR021" H 5350 3500 50  0001 C CNN
 F 1 "GNDD" H 5355 3577 50  0000 C CNN
 F 2 "" H 5350 3750 50  0000 C CNN
@@
 	5350 3500 5350 3450
 $Comp
-L C_Small C?
+L C_Small C4
 U 1 1 57A62CB7
 P 6050 3600
-F 0 "C?" H 6142 3646 50  0000 L CNN
+F 0 "C4" H 6142 3646 50  0000 L CNN
 F 1 "100uF 16V" H 6142 3555 50  0000 L CNN
 F 2 "" H 6050 3600 50  0000 C CNN
@@
 $EndComp
 $Comp
-L GNDD #PWR?
+L GNDD #PWR022
 U 1 1 57A62CBD
 P 6050 3750
-F 0 "#PWR?" H 6050 3500 50  0001 C CNN
+F 0 "#PWR022" H 6050 3500 50  0001 C CNN
 F 1 "GNDD" H 6055 3577 50  0000 C CNN
 F 2 "" H 6050 3750 50  0000 C CNN
@@
 Connection ~ 5350 3450
 $Comp
-L C_Small C?
+L C_Small C2
 U 1 1 57A62E19
 P 4850 4050
-F 0 "C?" H 4942 4096 50  0000 L CNN
+F 0 "C2" H 4942 4096 50  0000 L CNN
 F 1 "470nF" H 4942 4005 50  0000 L CNN
 F 2 "" H 4850 4050 50  0000 C CNN
@@
 $EndComp
 $Comp
-L GNDD #PWR?
+L GNDD #PWR023
 U 1 1 57A62E1F
 P 4850 4200
-F 0 "#PWR?" H 4850 3950 50  0001 C CNN
+F 0 "#PWR023" H 4850 3950 50  0001 C CNN
 F 1 "GNDD" H 4855 4027 50  0000 C CNN
 F 2 "" H 4850 4200 50  0000 C CNN
@@
 	4850 3800 4850 3950
 $Comp
-L PWR_FLAG #FLG?
+L PWR_FLAG #FLG024
 U 1 1 57A63012
 P 3050 3650
-F 0 "#FLG?" H 3050 3745 50  0001 C CNN
+F 0 "#FLG024" H 3050 3745 50  0001 C CNN
 F 1 "PWR_FLAG" H 3050 3873 50  0000 C CNN
 F 2 "" H 3050 3650 50  0000 C CNN
@@
 $EndComp
 $Comp
-L PWR_FLAG #FLG?
+L PWR_FLAG #FLG025
 U 1 1 57A63052
 P 3050 3450
-F 0 "#FLG?" H 3050 3545 50  0001 C CNN
+F 0 "#FLG025" H 3050 3545 50  0001 C CNN
 F 1 "PWR_FLAG" H 3050 3674 50  0000 C CNN
 F 2 "" H 3050 3450 50  0000 C CNN
@@
 	3350 3750 3600 3750
 $Comp
-L +5VA #PWR?
+L +5VA #PWR026
 U 1 1 57A630DE
 P 7100 3300
-F 0 "#PWR?" H 7100 3150 50  0001 C CNN
+F 0 "#PWR026" H 7100 3150 50  0001 C CNN
 F 1 "+5VA" H 7115 3473 50  0000 C CNN
 F 2 "" H 7100 3300 50  0000 C CNN
@@
 $EndComp
 $Comp
-L +5VD #PWR?
+L +5VD #PWR027
 U 1 1 57A63107
 P 6550 3300
-F 0 "#PWR?" H 6550 3150 50  0001 C CNN
+F 0 "#PWR027" H 6550 3150 50  0001 C CNN
 F 1 "+5VD" H 6565 3473 50  0000 C CNN
 F 2 "" H 6550 3300 50  0000 C CNN
@@
 Connection ~ 6050 3450
 $Comp
-L R_Small R?
+L R_Small R2
 U 1 1 57A633D8
 P 6850 3450
-F 0 "R?" V 7046 3450 50  0000 C CNN
-F 1 "0R" V 6955 3450 50  0000 C CNN
+F 0 "R2" V 7046 3450 50  0000 C CNN
+F 1 "0R/BEAD" V 6955 3450 50  0000 C CNN
 F 2 "" H 6850 3450 50  0000 C CNN
 F 3 "" H 6850 3450 50  0000 C CNN
@@
 	7100 3450 7100 3300
 $Comp
-L GNDD #PWR?
+L GNDD #PWR028
 U 1 1 57A63878
 P 7350 4500
-F 0 "#PWR?" H 7350 4250 50  0001 C CNN
+F 0 "#PWR028" H 7350 4250 50  0001 C CNN
 F 1 "GNDD" H 7355 4327 50  0000 C CNN
 F 2 "" H 7350 4500 50  0000 C CNN
@@
 Connection ~ 6700 3450
 $Comp
-L +3.3V #PWR?
+L +3.3V #PWR029
 U 1 1 57A63913
 P 8150 4100
-F 0 "#PWR?" H 8150 3950 50  0001 C CNN
+F 0 "#PWR029" H 8150 3950 50  0001 C CNN
 F 1 "+3.3V" H 8165 4273 50  0000 C CNN
 F 2 "" H 8150 4100 50  0000 C CNN
@@
 	7350 4500 7350 4450
 $Comp
-L C_Small C?
+L C_Small C6
 U 1 1 57A639D9
 P 8150 4300
-F 0 "C?" H 8242 4346 50  0000 L CNN
+F 0 "C6" H 8242 4346 50  0000 L CNN
 F 1 "10uF" H 8242 4255 50  0000 L CNN
 F 2 "" H 8150 4300 50  0000 C CNN
@@
 	6700 4450 8150 4450
 $Comp
-L C_Small C?
+L C_Small C5
 U 1 1 57A63B2D
 P 6700 4300
-F 0 "C?" H 6792 4346 50  0000 L CNN
+F 0 "C5" H 6792 4346 50  0000 L CNN
 F 1 "10uF" H 6792 4255 50  0000 L CNN
 F 2 "" H 6700 4300 50  0000 C CNN
@@
 Connection ~ 7350 4450
 Connection ~ 6700 4100
+Connection ~ 3050 3450
+Connection ~ 3050 3650
+NoConn ~ 4750 3800
+$Comp
+L PWR_FLAG #FLG030
+U 1 1 57A8371C
+P 7100 3450
+F 0 "#FLG030" H 7100 3545 50  0001 C CNN
+F 1 "PWR_FLAG" V 7100 3628 50  0000 L CNN
+F 2 "" H 7100 3450 50  0000 C CNN
+F 3 "" H 7100 3450 50  0000 C CNN
+	1    7100 3450
+	0    1    1    0
+$EndComp
 $EndSCHEMATC

Commit message: Footprints assigned, netlist generated - ready for layout
Parts:
- C1, C3, C5, C6: footprint (none) -> Capacitors_SMD:C_1210
- C2: footprint (none) -> Capacitors_SMD:C_0805
- C4: footprint (none) -> sictroller:C_6x5
- J5: renamed from CON1; footprint (none) -> Connect:BARREL_JACK
- R2: footprint (none) -> Resistors_SMD:R_0805
- U1: footprint (none) -> sictroller:V78-500-SMT
- U2: footprint SOT-23 -> TO_SOT_Packages_SMD:SOT-23
Changed lines of the file:
@@
 $EndDescr
 $Comp
-L BARREL_JACK CON1
+L BARREL_JACK J5
 U 1 1 57A588D1
 P 2600 3550
-F 0 "CON1" H 2581 3875 50  0000 C CNN
+F 0 "J5" H 2581 3875 50  0000 C CNN
 F 1 "BARREL_JACK" H 2581 3784 50  0000 C CNN
-F 2 "" H 2600 3550 50  0000 C CNN
+F 2 "Connect:BARREL_JACK" H 2600 3550 50  0001 C CNN
 F 3 "" H 2600 3550 50  0000 C CNN
 	1    2600 3550
@@
 F 0 "U2" H 7350 4558 50  0000 C CNN
 F 1 "APE8865N-33-HF-3" H 7350 4467 50  0000 C CNN
-F 2 "SOT-23" H 7350 4376 50  0000 C CIN
+F 2 "TO_SOT_Packages_SMD:SOT-23" H 7350 4376 50  0000 C CIN
 F 3 "" H 7350 4150 50  0000 C CNN
 	1    7350 4150
@@
 F 0 "U1" H 4700 3687 60  0000 C CNN
 F 1 "V7805-500-SMT" H 4700 3581 60  0000 C CNN
-F 2 "" H 4700 3400 60  0001 C CNN
+F 2 "sictroller:V78-500-SMT" H 4700 3400 60  0001 C CNN
 F 3 "" H 4700 3400 60  0001 C CNN
 	1    4700 3400
@@
 F 0 "C1" H 3692 3646 50  0000 L CNN
 F 1 "10uF 50V" H 3692 3555 50  0000 L CNN
-F 2 "" H 3600 3600 50  0000 C CNN
+F 2 "Capacitors_SMD:C_1210" H 3600 3600 50  0001 C CNN
 F 3 "" H 3600 3600 50  0000 C CNN
 	1    3600 3600
@@
 F 0 "C3" H 5442 3646 50  0000 L CNN
 F 1 "22uF 16V" H 5442 3555 50  0000 L CNN
-F 2 "" H 5350 3600 50  0000 C CNN
+F 2 "Capacitors_SMD:C_1210" H 5350 3600 50  0001 C CNN
 F 3 "" H 5350 3600 50  0000 C CNN
 	1    5350 3600
@@
 F 0 "C4" H 6142 3646 50  0000 L CNN
 F 1 "100uF 16V" H 6142 3555 50  0000 L CNN
-F 2 "" H 6050 3600 50  0000 C CNN
+F 2 "sictroller:C_6x5" H 6050 3600 50  0001 C CNN
 F 3 "" H 6050 3600 50  0000 C CNN
 	1    6050 3600
@@
 F 0 "C2" H 4942 4096 50  0000 L CNN
 F 1 "470nF" H 4942 4005 50  0000 L CNN
-F 2 "" H 4850 4050 50  0000 C CNN
+F 2 "Capacitors_SMD:C_0805" H 4850 4050 50  0001 C CNN
 F 3 "" H 4850 4050 50  0000 C CNN
 	1    4850 4050
@@
 F 0 "R2" V 7046 3450 50  0000 C CNN
 F 1 "0R/BEAD" V 6955 3450 50  0000 C CNN
-F 2 "" H 6850 3450 50  0000 C CNN
+F 2 "Resistors_SMD:R_0805" H 6850 3450 50  0001 C CNN
 F 3 "" H 6850 3450 50  0000 C CNN
 	1    6850 3450
@@
 F 0 "C6" H 8242 4346 50  0000 L CNN
 F 1 "10uF" H 8242 4255 50  0000 L CNN
-F 2 "" H 8150 4300 50  0000 C CNN
+F 2 "Capacitors_SMD:C_1210" H 8150 4300 50  0001 C CNN
 F 3 "" H 8150 4300 50  0000 C CNN
 	1    8150 4300
@@
 F 0 "C5" H 6792 4346 50  0000 L CNN
 F 1 "10uF" H 6792 4255 50  0000 L CNN
-F 2 "" H 6700 4300 50  0000 C CNN
+F 2 "Capacitors_SMD:C_1210" H 6700 4300 50  0001 C CNN
 F 3 "" H 6700 4300 50  0000 C CNN
 	1    6700 4300

Commit message: More aux pins, SKUs for some components
Parts:
- C2: footprint Capacitors_SMD:C_0805 -> Capacitors_SMD:C_0603
- J5: footprint Connect:BARREL_JACK -> sictroller:PJ-102B; SKU (none) -> CP-102B-ND
- R2: footprint Resistors_SMD:R_0805 -> Resistors_SMD:R_0603
- U1: SKU (none) -> 490-V7805-500-SMT-TR; Supplier (none) -> Mouser
Changed lines of the file:
@@
 F 0 "J5" H 2581 3875 50  0000 C CNN
 F 1 "BARREL_JACK" H 2581 3784 50  0000 C CNN
-F 2 "Connect:BARREL_JACK" H 2600 3550 50  0001 C CNN
+F 2 "sictroller:PJ-102B" H 2600 3550 50  0001 C CNN
 F 3 "" H 2600 3550 50  0000 C CNN
+F 4 "CP-102B-ND" H 2600 3550 60  0001 C CNN "SKU"
 	1    2600 3550
 	1    0    0    -1
@@
 F 2 "sictroller:V78-500-SMT" H 4700 3400 60  0001 C CNN
 F 3 "" H 4700 3400 60  0001 C CNN
+F 4 "Mouser" H 4700 3400 60  0001 C CNN "Supplier"
+F 5 "490-V7805-500-SMT-TR" H 4700 3400 60  0001 C CNN "SKU"
 	1    4700 3400
 	1    0    0    -1
@@
 F 0 "C2" H 4942 4096 50  0000 L CNN
 F 1 "470nF" H 4942 4005 50  0000 L CNN
-F 2 "Capacitors_SMD:C_0805" H 4850 4050 50  0001 C CNN
+F 2 "Capacitors_SMD:C_0603" H 4850 4050 50  0001 C CNN
 F 3 "" H 4850 4050 50  0000 C CNN
 	1    4850 4050
@@
 F 0 "R2" V 7046 3450 50  0000 C CNN
 F 1 "0R/BEAD" V 6955 3450 50  0000 C CNN
-F 2 "Resistors_SMD:R_0805" H 6850 3450 50  0001 C CNN
+F 2 "Resistors_SMD:R_0603" H 6850 3450 50  0001 C CNN
 F 3 "" H 6850 3450 50  0000 C CNN
 	1    6850 3450
