File: CGD15FB45P1.sch (KiCad schematic (older format))
At the start: 10 parts

Commit message: V0 schematic complete (?)
Parts:
- removed R?: 10k, symbol R_Small
- removed R? (x2): 5k1, symbol R_Small
- added C3: 1uF, symbol C_Small
- added U2: 74LVC2G04, symbol 74LVC2G04
- gave numbers to parts that had none: 7
Connections:
- net FLT_DESAT is gone; now on net PWR_RDY: R3.7
- net +3V3: now also C3.1, U2.5 (VCC), U2.5 (VCC)
- net FLT_DESAT_TTL: now also U2.1
- net FLT_OTP_TTL: now also U2.3
- net ~PWR_RESET: now also R4.2
- net FLT_OTP: no longer names the net of R3.6
- net GNDD renamed GND
- net GND: now also C3.2, U2.2 (GND), U2.2 (GND)
- new net ~FLT_DESAT: U2.6
- new net ~FLT_OTP: U2.4
- no-connect marks 0 -> 3
Other:
- moved on the sheet: J3, R3, R5

Commit message: Annotate, fix schematic DRC, footprint for DIMM100
Parts:
- renumbered C1 to C25, C2 to C26, C3 to C27, J3 to J6, R3 to R37, R4 to R38, R5 to R39, U1 to U6, U2 to U7
Changed lines of the file:
@@
 $EndDescr
 $Comp
-L GNDD #PWR012
+L GNDD #PWR067
 U 1 1 57A1908E
 P 7350 5850
-F 0 "#PWR012" H 7350 5600 50  0001 C CNN
+F 0 "#PWR067" H 7350 5600 50  0001 C CNN
 F 1 "GNDD" H 7350 5700 50  0000 C CNN
 F 2 "" H 7350 5850 50  0000 C CNN
@@
 $EndComp
 $Comp
-L 74LVC8T245 U1
+L 74LVC8T245 U6
 U 1 1 57A19094
 P 5350 4950
-F 0 "U1" H 5150 5900 60  0000 L CNN
+F 0 "U6" H 5150 5900 60  0000 L CNN
 F 1 "74LVC8T245" H 5150 4100 60  0000 L CNN
 F 2 "" H 5350 4250 60  0000 C CNN
@@
 $EndComp
 $Comp
-L +5VD #PWR013
+L +5VD #PWR068
 U 1 1 57A1909B
 P 5850 3850
-F 0 "#PWR013" H 5850 3700 50  0001 C CNN
+F 0 "#PWR068" H 5850 3700 50  0001 C CNN
 F 1 "+5VD" H 5850 3990 50  0000 C CNN
 F 2 "" H 5850 3850 50  0000 C CNN
@@
 PWM_CL
 $Comp
-L R_Small R4
+L R_Small R38
 U 1 1 57A190B9
 P 3300 4850
-F 0 "R4" H 3330 4870 50  0000 L CNN
+F 0 "R38" H 3330 4870 50  0000 L CNN
 F 1 "10k" H 3330 4810 50  0000 L CNN
 F 2 "" H 3300 4850 50  0000 C CNN
@@
 FLT_DESAT_TTL
 $Comp
-L CONN_02X13 J3
+L CONN_02X13 J6
 U 1 1 57A190E8
 P 7100 5050
-F 0 "J3" H 7100 5750 50  0000 C CNN
+F 0 "J6" H 7100 5750 50  0000 C CNN
 F 1 "CONN_02X13" V 7100 5050 50  0000 C CNN
 F 2 "" H 7100 3900 50  0000 C CNN
@@
 PWM_BH
 $Comp
-L +15V #PWR014
+L +15V #PWR069
 U 1 1 57A190F2
 P 6650 5650
-F 0 "#PWR014" H 6650 5500 50  0001 C CNN
+F 0 "#PWR069" H 6650 5500 50  0001 C CNN
 F 1 "+15V" H 6650 5790 50  0000 C CNN
 F 2 "" H 6650 5650 50  0000 C CNN
@@
 FLT_OTP_TTL
 $Comp
-L C_Small C2
+L C_Small C26
 U 1 1 57A190F9
 P 6000 4050
-F 0 "C2" H 6010 4120 50  0000 L CNN
+F 0 "C26" H 6010 4120 50  0000 L CNN
 F 1 "1uF" H 6010 3970 50  0000 L CNN
 F 2 "" H 6000 4050 50  0000 C CNN
@@
 $EndComp
 $Comp
-L GNDD #PWR015
+L GNDD #PWR070
 U 1 1 57A19106
 P 4650 4150
-F 0 "#PWR015" H 4650 3900 50  0001 C CNN
+F 0 "#PWR070" H 4650 3900 50  0001 C CNN
 F 1 "GNDD" H 4650 4000 50  0000 C CNN
 F 2 "" H 4650 4150 50  0000 C CNN
@@
 $EndComp
 $Comp
-L GNDD #PWR016
+L GNDD #PWR071
 U 1 1 57A1910C
 P 6000 4150
-F 0 "#PWR016" H 6000 3900 50  0001 C CNN
+F 0 "#PWR071" H 6000 3900 50  0001 C CNN
 F 1 "GNDD" H 6000 4000 50  0000 C CNN
 F 2 "" H 6000 4150 50  0000 C CNN
@@
 PWM_BL
 $Comp
-L +3.3V #PWR017
+L +3.3V #PWR072
 U 1 1 57A19125
 P 3300 4700
-F 0 "#PWR017" H 3300 4550 50  0001 C CNN
+F 0 "#PWR072" H 3300 4550 50  0001 C CNN
 F 1 "+3.3V" H 3300 4840 50  0000 C CNN
 F 2 "" H 3300 4700 50  0000 C CNN
@@
 PWR_RDY_TTL
 $Comp
-L R_Small R5
+L R_Small R39
 U 1 1 57A1913E
 P 4150 2000
-F 0 "R5" H 4180 2020 50  0000 L CNN
+F 0 "R39" H 4180 2020 50  0000 L CNN
 F 1 "5k1" H 4180 1960 50  0000 L CNN
 F 2 "" H 4150 2000 50  0000 C CNN
@@
 	4150 1850 4750 1850
 $Comp
-L GNDD #PWR018
+L GNDD #PWR073
 U 1 1 57A19193
 P 4950 5900
-F 0 "#PWR018" H 4950 5650 50  0001 C CNN
+F 0 "#PWR073" H 4950 5650 50  0001 C CNN
 F 1 "GNDD" H 4950 5750 50  0000 C CNN
 F 2 "" H 4950 5900 50  0000 C CNN
@@
 PWR_RDY
 $Comp
-L R_ARRAY_8_10 R3
+L R_ARRAY_8_10 R37
 U 1 1 57A19112
 P 3000 2100
-F 0 "R3" H 2800 1800 60  0000 C CNN
+F 0 "R37" H 2800 1800 60  0000 C CNN
 F 1 "10k" H 3300 1800 60  0000 C CNN
 F 2 "" H 3100 1950 60  0000 C CNN
@@
 $EndComp
 $Comp
-L +3.3V #PWR019
+L +3.3V #PWR074
 U 1 1 57A19100
 P 4950 3850
-F 0 "#PWR019" H 4950 3700 50  0001 C CNN
+F 0 "#PWR074" H 4950 3700 50  0001 C CNN
 F 1 "+3.3V" H 4950 3990 50  0000 C CNN
 F 2 "" H 4950 3850 50  0000 C CNN
@@
 $EndComp
 $Comp
-L C_Small C1
+L C_Small C25
 U 1 1 57A190A6
 P 4650 4050
-F 0 "C1" H 4660 4120 50  0000 L CNN
+F 0 "C25" H 4660 4120 50  0000 L CNN
 F 1 "1uF" H 4660 3970 50  0000 L CNN
 F 2 "" H 4650 4050 50  0000 C CNN
@@
 Connection ~ 6850 5650
 $Comp
-L GNDD #PWR020
+L GNDD #PWR075
 U 1 1 57A1911A
 P 2550 2300
-F 0 "#PWR020" H 2550 2050 50  0001 C CNN
+F 0 "#PWR075" H 2550 2050 50  0001 C CNN
 F 1 "GNDD" H 2550 2150 50  0000 C CNN
 F 2 "" H 2550 2300 50  0000 C CNN
@@
 	4150 2200 3300 2200
 $Comp
-L 74LVC2G04 U2
+L 74LVC2G04 U7
 U 1 1 57A2374F
 P 6350 2200
-F 0 "U2" H 6450 2400 50  0000 C CNN
+F 0 "U7" H 6450 2400 50  0000 C CNN
 F 1 "74LVC2G04" H 6600 2300 50  0000 C CNN
 F 2 "" H 6350 2200 50  0000 C CNN
@@
 $EndComp
 $Comp
-L 74LVC2G04 U2
+L 74LVC2G04 U7
 U 2 1 57A23A29
 P 6350 3000
-F 0 "U2" H 6350 3315 50  0000 C CNN
+F 0 "U7" H 6350 3315 50  0000 C CNN
 F 1 "74LVC2G04" H 6350 3224 50  0000 C CNN
 F 2 "" H 6350 3000 50  0000 C CNN
@@
 $EndComp
 $Comp
-L GNDD #PWR021
+L GNDD #PWR076
 U 1 1 57A23C37
 P 6300 2400
-F 0 "#PWR021" H 6300 2150 50  0001 C CNN
+F 0 "#PWR076" H 6300 2150 50  0001 C CNN
 F 1 "GNDD" H 6300 2250 50  0000 C CNN
 F 2 "" H 6300 2400 50  0000 C CNN
@@
 	6300 2400 6300 2300
 $Comp
-L +3.3V #PWR022
+L +3.3V #PWR077
 U 1 1 57A23E25
 P 6300 1450
-F 0 "#PWR022" H 6300 1300 50  0001 C CNN
+F 0 "#PWR077" H 6300 1300 50  0001 C CNN
 F 1 "+3.3V" H 6300 1590 50  0000 C CNN
 F 2 "" H 6300 1450 50  0000 C CNN
@@
 	6300 1450 6300 2100
 $Comp
-L GNDD #PWR023
+L GNDD #PWR078
 U 1 1 57A244F4
 P 6600 1700
-F 0 "#PWR023" H 6600 1450 50  0001 C CNN
+F 0 "#PWR078" H 6600 1450 50  0001 C CNN
 F 1 "GNDD" H 6600 1550 50  0000 C CNN
 F 2 "" H 6600 1700 50  0000 C CNN
@@
 	6600 1500 6600 1450
 $Comp
-L C_Small C3
+L C_Small C27
 U 1 1 57A244FB
 P 6600 1600
-F 0 "C3" H 6610 1670 50  0000 L CNN
+F 0 "C27" H 6610 1670 50  0000 L CNN
 F 1 "1uF" H 6610 1520 50  0000 L CNN
 F 2 "" H 6600 1600 50  0000 C CNN

Commit message: Footprints assigned, netlist generated - ready for layout
Parts:
- C25, C26, C27: footprint (none) -> Capacitors_SMD:C_0805
- J12: renamed from J6; footprint (none) -> Connect:IDC_Header_Straight_26pins
- R37: value 10k -> 745C101103 (10k); footprint (none) -> Resistors_SMD:R_Array_Convex_5x1206
- R38, R39: footprint (none) -> Resistors_SMD:R_0805
- U6: footprint (none) -> Housings_SSOP:TSSOP-24_4.4x7.8mm_Pitch0.65mm
- U7: footprint (none) -> TO_SOT_Packages_SMD:TSOT-6-MK06A
Changed lines of the file:
@@
 F 0 "U6" H 5150 5900 60  0000 L CNN
 F 1 "74LVC8T245" H 5150 4100 60  0000 L CNN
-F 2 "" H 5350 4250 60  0000 C CNN
+F 2 "Housings_SSOP:TSSOP-24_4.4x7.8mm_Pitch0.65mm" H 5350 4250 60  0001 C CNN
 F 3 "" H 5350 4250 60  0000 C CNN
 	1    5350 4950
@@
 F 0 "R38" H 3330 4870 50  0000 L CNN
 F 1 "10k" H 3330 4810 50  0000 L CNN
-F 2 "" H 3300 4850 50  0000 C CNN
+F 2 "Resistors_SMD:R_0805" H 3300 4850 50  0001 C CNN
 F 3 "" H 3300 4850 50  0000 C CNN
 	1    3300 4850
@@
 FLT_DESAT_TTL
 $Comp
-L CONN_02X13 J6
+L CONN_02X13 J12
 U 1 1 57A190E8
 P 7100 5050
-F 0 "J6" H 7100 5750 50  0000 C CNN
+F 0 "J12" H 7100 5750 50  0000 C CNN
 F 1 "CONN_02X13" V 7100 5050 50  0000 C CNN
-F 2 "" H 7100 3900 50  0000 C CNN
+F 2 "Connect:IDC_Header_Straight_26pins" H 7100 3900 50  0001 C CNN
 F 3 "" H 7100 3900 50  0000 C CNN
 	1    7100 5050
@@
 F 0 "C26" H 6010 4120 50  0000 L CNN
 F 1 "1uF" H 6010 3970 50  0000 L CNN
-F 2 "" H 6000 4050 50  0000 C CNN
+F 2 "Capacitors_SMD:C_0805" H 6000 4050 50  0001 C CNN
 F 3 "" H 6000 4050 50  0000 C CNN
 	1    6000 4050
@@
 F 0 "R39" H 4180 2020 50  0000 L CNN
 F 1 "5k1" H 4180 1960 50  0000 L CNN
-F 2 "" H 4150 2000 50  0000 C CNN
+F 2 "Resistors_SMD:R_0805" H 4150 2000 50  0001 C CNN
 F 3 "" H 4150 2000 50  0000 C CNN
 	1    4150 2000
@@
 P 3000 2100
 F 0 "R37" H 2800 1800 60  0000 C CNN
-F 1 "10k" H 3300 1800 60  0000 C CNN
-F 2 "" H 3100 1950 60  0000 C CNN
+F 1 "745C101103 (10k)" H 3300 1800 60  0000 C CNN
+F 2 "Resistors_SMD:R_Array_Convex_5x1206" H 3100 1950 60  0001 C CNN
 F 3 "" H 3100 1950 60  0000 C CNN
 	1    3000 2100
@@
 F 0 "C25" H 4660 4120 50  0000 L CNN
 F 1 "1uF" H 4660 3970 50  0000 L CNN
-F 2 "" H 4650 4050 50  0000 C CNN
+F 2 "Capacitors_SMD:C_0805" H 4650 4050 50  0001 C CNN
 F 3 "" H 4650 4050 50  0000 C CNN
 	1    4650 4050
@@
 F 0 "U7" H 6450 2400 50  0000 C CNN
 F 1 "74LVC2G04" H 6600 2300 50  0000 C CNN
-F 2 "" H 6350 2200 50  0000 C CNN
+F 2 "TO_SOT_Packages_SMD:TSOT-6-MK06A" H 6350 2200 50  0001 C CNN
 F 3 "" H 6350 2200 50  0000 C CNN
 	1    6350 2200
@@
 F 0 "U7" H 6350 3315 50  0000 C CNN
 F 1 "74LVC2G04" H 6350 3224 50  0000 C CNN
-F 2 "" H 6350 3000 50  0000 C CNN
+F 2 "TO_SOT_Packages_SMD:TSOT-6-MK06A" H 6350 3000 50  0001 C CNN
 F 3 "" H 6350 3000 50  0000 C CNN
 	2    6350 3000
@@
 F 0 "C27" H 6610 1670 50  0000 L CNN
 F 1 "1uF" H 6610 1520 50  0000 L CNN
-F 2 "" H 6600 1600 50  0000 C CNN
+F 2 "Capacitors_SMD:C_0805" H 6600 1600 50  0001 C CNN
 F 3 "" H 6600 1600 50  0000 C CNN
 	1    6600 1600

Commit message: More aux pins, SKUs for some components
Parts:
- C25, C26, C27: footprint Capacitors_SMD:C_0805 -> Capacitors_SMD:C_0603
- R37: SKU (none) -> 745C101103JPCT-ND
- R38, R39: footprint Resistors_SMD:R_0805 -> Resistors_SMD:R_0603
Changed lines of the file:
@@
 F 0 "R38" H 3330 4870 50  0000 L CNN
 F 1 "10k" H 3330 4810 50  0000 L CNN
-F 2 "Resistors_SMD:R_0805" H 3300 4850 50  0001 C CNN
+F 2 "Resistors_SMD:R_0603" H 3300 4850 50  0001 C CNN
 F 3 "" H 3300 4850 50  0000 C CNN
 	1    3300 4850
@@
 F 0 "C26" H 6010 4120 50  0000 L CNN
 F 1 "1uF" H 6010 3970 50  0000 L CNN
-F 2 "Capacitors_SMD:C_0805" H 6000 4050 50  0001 C CNN
+F 2 "Capacitors_SMD:C_0603" H 6000 4050 50  0001 C CNN
 F 3 "" H 6000 4050 50  0000 C CNN
 	1    6000 4050
@@
 F 0 "R39" H 4180 2020 50  0000 L CNN
 F 1 "5k1" H 4180 1960 50  0000 L CNN
-F 2 "Resistors_SMD:R_0805" H 4150 2000 50  0001 C CNN
+F 2 "Resistors_SMD:R_0603" H 4150 2000 50  0001 C CNN
 F 3 "" H 4150 2000 50  0000 C CNN
 	1    4150 2000
@@
 F 2 "Resistors_SMD:R_Array_Convex_5x1206" H 3100 1950 60  0001 C CNN
 F 3 "" H 3100 1950 60  0000 C CNN
+F 4 "745C101103JPCT-ND" H 3000 2100 60  0001 C CNN "SKU"
 	1    3000 2100
 	1    0    0    -1
@@
 F 0 "C25" H 4660 4120 50  0000 L CNN
 F 1 "1uF" H 4660 3970 50  0000 L CNN
-F 2 "Capacitors_SMD:C_0805" H 4650 4050 50  0001 C CNN
+F 2 "Capacitors_SMD:C_0603" H 4650 4050 50  0001 C CNN
 F 3 "" H 4650 4050 50  0000 C CNN
 	1    4650 4050
@@
 F 0 "C27" H 6610 1670 50  0000 L CNN
 F 1 "1uF" H 6610 1520 50  0000 L CNN
-F 2 "Capacitors_SMD:C_0805" H 6600 1600 50  0001 C CNN
+F 2 "Capacitors_SMD:C_0603" H 6600 1600 50  0001 C CNN
 F 3 "" H 6600 1600 50  0000 C CNN
 	1    6600 1600
