File: feedback.sch (KiCad schematic (older format))
At the start: 59 parts, among them J10 CONN_01X02, J11 RINGTERM, J12 RINGTERM, J4 RINGTERM, J5 RINGTERM, J6 RINGTERM, J7 CONN_01X02, J8 RINGTERM, J9 RINGTERM, Q1 CSD17483F4, U8 ADUM5241, U9 MAX6691

Commit message: Footprints assigned for all except halfbridge-driver
Parts:
- C39, C40, C49, C50, C52, C53, C54, C55, C56: footprint Capacitors_SMD:C_0603 -> Capacitors_SMD:C_0402
- I1, I2, I3: footprint (none) -> sictroller:ACS770
- J10, J7: footprint sictroller:Molex-SL-2POS-RA -> Connectors_Molex:Molex_PicoBlade_53261-0271
- J11, J12, J4, J5, J6, J8, J9: footprint (none) -> sictroller:B6A-PCB
- Q1: footprint (none) -> sictroller:FEMTOFET_YJC_YJJ
- R24, R29, R38, R39, R40, R41, R42, R43, R44, R45, R46: footprint Resistors_SMD:R_0603 -> Resistors_SMD:R_0402
- TH1: value THERMISTOR -> NCP15XW153J03RC; footprint (none) -> Resistors_SMD:R_0402
- U8: footprint (none) -> Housings_SOIC:SOIC-8_3.9x4.9mm_Pitch1.27mm
- U9: footprint (none) -> Housings_SSOP:MSOP-10_3x3mm_Pitch0.5mm
Other:
- note added: "Also, main high power external connections are here."
- note removed: "Also, main high power external\nconnections are here."
Changed lines of the file:
@@
 F 0 "R24" H 9950 1750 50  0000 C CNN
 F 1 "1.8K" H 9950 1850 50  0000 C CNN
-F 2 "Resistors_SMD:R_0603" H 9800 1750 50  0001 C CNN
+F 2 "Resistors_SMD:R_0402" H 9800 1750 50  0001 C CNN
 F 3 "" H 9800 1750 50  0000 C CNN
 	1    9800 1750
@@
 F 0 "R29" H 9950 2100 50  0000 C CNN
 F 1 "3.3K" H 9950 2200 50  0000 C CNN
-F 2 "Resistors_SMD:R_0603" H 9800 2100 50  0001 C CNN
+F 2 "Resistors_SMD:R_0402" H 9800 2100 50  0001 C CNN
 F 3 "" H 9800 2100 50  0000 C CNN
 	1    9800 2100
@@
 F 0 "C40" H 10100 2100 50  0000 L CNN
 F 1 "1nF" H 10100 2000 50  0000 L CNN
-F 2 "Capacitors_SMD:C_0603" H 10000 2100 50  0001 C CNN
+F 2 "Capacitors_SMD:C_0402" H 10000 2100 50  0001 C CNN
 F 3 "" H 10000 2100 50  0000 C CNN
 	1    10000 2100
@@
 F 0 "R38" H 9950 3550 50  0000 C CNN
 F 1 "1.8K" H 9950 3650 50  0000 C CNN
-F 2 "Resistors_SMD:R_0603" H 9800 3550 50  0001 C CNN
+F 2 "Resistors_SMD:R_0402" H 9800 3550 50  0001 C CNN
 F 3 "" H 9800 3550 50  0000 C CNN
 	1    9800 3550
@@
 F 0 "R39" H 9950 3900 50  0000 C CNN
 F 1 "3.3K" H 9950 4000 50  0000 C CNN
-F 2 "Resistors_SMD:R_0603" H 9800 3900 50  0001 C CNN
+F 2 "Resistors_SMD:R_0402" H 9800 3900 50  0001 C CNN
 F 3 "" H 9800 3900 50  0000 C CNN
 	1    9800 3900
@@
 F 0 "C50" H 10100 3900 50  0000 L CNN
 F 1 "1nF" H 10100 3800 50  0000 L CNN
-F 2 "Capacitors_SMD:C_0603" H 10000 3900 50  0001 C CNN
+F 2 "Capacitors_SMD:C_0402" H 10000 3900 50  0001 C CNN
 F 3 "" H 10000 3900 50  0000 C CNN
 	1    10000 3900
@@
 F 0 "R42" H 9950 5350 50  0000 C CNN
 F 1 "1.8K" H 9950 5450 50  0000 C CNN
-F 2 "Resistors_SMD:R_0603" H 9800 5350 50  0001 C CNN
+F 2 "Resistors_SMD:R_0402" H 9800 5350 50  0001 C CNN
 F 3 "" H 9800 5350 50  0000 C CNN
 	1    9800 5350
@@
 F 0 "R44" H 9950 5700 50  0000 C CNN
 F 1 "3.3K" H 9950 5800 50  0000 C CNN
-F 2 "Resistors_SMD:R_0603" H 9800 5700 50  0001 C CNN
+F 2 "Resistors_SMD:R_0402" H 9800 5700 50  0001 C CNN
 F 3 "" H 9800 5700 50  0000 C CNN
 	1    9800 5700
@@
 F 0 "C56" H 10100 5700 50  0000 L CNN
 F 1 "1nF" H 10100 5600 50  0000 L CNN
-F 2 "Capacitors_SMD:C_0603" H 10000 5700 50  0001 C CNN
+F 2 "Capacitors_SMD:C_0402" H 10000 5700 50  0001 C CNN
 F 3 "" H 10000 5700 50  0000 C CNN
 	1    10000 5700
@@
 F 0 "J7" H 1478 5441 50  0000 L CNN
 F 1 "CONN_01X02" H 1478 5350 50  0000 L CNN
-F 2 "sictroller:Molex-SL-2POS-RA" H 1400 5400 50  0001 C CNN
+F 2 "Connectors_Molex:Molex_PicoBlade_53261-0271" H 1400 5400 50  0001 C CNN
 F 3 "" H 1400 5400 50  0000 C CNN
 	1    1400 5400
@@
 F 0 "I1" H 8900 1200 60  0000 C CNN
 F 1 "ACS770" H 8900 1500 60  0000 C CNN
-F 2 "" H 8900 1350 60  0001 C CNN
+F 2 "sictroller:ACS770" H 8900 1350 60  0001 C CNN
 F 3 "" H 8900 1350 60  0000 C CNN
 	1    8900 1350
@@
 F 0 "I2" H 8900 3000 60  0000 C CNN
 F 1 "ACS770" H 8900 3300 60  0000 C CNN
-F 2 "" H 8900 3150 60  0001 C CNN
+F 2 "sictroller:ACS770" H 8900 3150 60  0001 C CNN
 F 3 "" H 8900 3150 60  0000 C CNN
 	1    8900 3150
@@
 F 0 "I3" H 8900 4800 60  0000 C CNN
 F 1 "ACS770" H 8900 5100 60  0000 C CNN
-F 2 "" H 8900 4950 60  0001 C CNN
+F 2 "sictroller:ACS770" H 8900 4950 60  0001 C CNN
 F 3 "" H 8900 4950 60  0000 C CNN
 	1    8900 4950
@@
 F 0 "C39" H 9600 1200 50  0000 L CNN
 F 1 "0.1uF" H 9600 1100 50  0000 L CNN
-F 2 "Capacitors_SMD:C_0603" H 9500 1200 50  0001 C CNN
+F 2 "Capacitors_SMD:C_0402" H 9500 1200 50  0001 C CNN
 F 3 "" H 9500 1200 50  0000 C CNN
 	1    9500 1200
@@
 F 0 "C49" H 9600 3000 50  0000 L CNN
 F 1 "0.1uF" H 9600 2900 50  0000 L CNN
-F 2 "Capacitors_SMD:C_0603" H 9500 3000 50  0001 C CNN
+F 2 "Capacitors_SMD:C_0402" H 9500 3000 50  0001 C CNN
 F 3 "" H 9500 3000 50  0000 C CNN
 	1    9500 3000
@@
 F 0 "C53" H 9600 4800 50  0000 L CNN
 F 1 "0.1uF" H 9600 4700 50  0000 L CNN
-F 2 "Capacitors_SMD:C_0603" H 9500 4800 50  0001 C CNN
+F 2 "Capacitors_SMD:C_0402" H 9500 4800 50  0001 C CNN
 F 3 "" H 9500 4800 50  0000 C CNN
 	1    9500 4800
@@
 F 0 "J4" H 8100 1700 50  0000 C CNN
 F 1 "RINGTERM" V 8200 1600 50  0000 C CNN
-F 2 "" H 8100 1600 50  0001 C CNN
+F 2 "sictroller:B6A-PCB" H 8100 1600 50  0001 C CNN
 F 3 "" H 8100 1600 50  0000 C CNN
 	1    8100 1600
@@
 F 0 "J5" H 8100 3000 50  0000 C CNN
 F 1 "RINGTERM" V 8200 2900 50  0000 C CNN
-F 2 "" H 8100 2900 50  0001 C CNN
+F 2 "sictroller:B6A-PCB" H 8100 2900 50  0001 C CNN
 F 3 "" H 8100 2900 50  0000 C CNN
 	1    8100 2900
@@
 F 0 "J6" H 8100 4800 50  0000 C CNN
 F 1 "RINGTERM" V 8200 4700 50  0000 C CNN
-F 2 "" H 8100 4700 50  0001 C CNN
+F 2 "sictroller:B6A-PCB" H 8100 4700 50  0001 C CNN
 F 3 "" H 8100 4700 50  0000 C CNN
 	1    8100 4700
@@
 F 0 "J11" H 7950 6450 50  0000 C CNN
 F 1 "RINGTERM" V 8050 6350 50  0000 C CNN
-F 2 "" H 7950 6350 50  0001 C CNN
+F 2 "sictroller:B6A-PCB" H 7950 6350 50  0001 C CNN
 F 3 "" H 7950 6350 50  0000 C CNN
 	1    7950 6350
@@
 F 0 "J12" H 9200 6450 50  0000 C CNN
 F 1 "RINGTERM" V 9300 6350 50  0000 C CNN
-F 2 "" H 9200 6350 50  0001 C CNN
+F 2 "sictroller:B6A-PCB" H 9200 6350 50  0001 C CNN
 F 3 "" H 9200 6350 50  0000 C CNN
 	1    9200 6350
@@
 F 0 "U8" H 4590 4990 60  0000 C CNN
 F 1 "ADUM5241" H 5130 4990 60  0000 C CNN
-F 2 "" H 5850 4750 60  0001 C CNN
+F 2 "Housings_SOIC:SOIC-8_3.9x4.9mm_Pitch1.27mm" H 5850 4750 60  0001 C CNN
 F 3 "" H 5850 4750 60  0001 C CNN
 	1    4950 5350
@@
 F 0 "U9" H 3000 5350 60  0000 C CNN
 F 1 "MAX6691" H 3500 5350 60  0000 C CNN
-F 2 "" H 3200 5550 60  0001 C CNN
+F 2 "Housings_SSOP:MSOP-10_3x3mm_Pitch0.5mm" H 3200 5550 60  0001 C CNN
 F 3 "" H 3200 5550 60  0001 C CNN
 	1    3200 5550
@@
 F 0 "C52" H 4850 4800 50  0000 L CNN
 F 1 "0.1uF" H 4850 4700 50  0000 L CNN
-F 2 "Capacitors_SMD:C_0603" H 4750 4800 50  0001 C CNN
+F 2 "Capacitors_SMD:C_0402" H 4750 4800 50  0001 C CNN
 F 3 "" H 4750 4800 50  0000 C CNN
 	1    4750 4800
@@
 F 0 "R46" H 3400 5850 50  0000 C CNN
 F 1 "2.7K" H 3400 5950 50  0000 C CNN
-F 2 "Resistors_SMD:R_0603" H 3250 5850 50  0001 C CNN
+F 2 "Resistors_SMD:R_0402" H 3250 5850 50  0001 C CNN
 F 3 "" H 3250 5850 50  0000 C CNN
 	1    3250 5850
@@
 F 0 "R40" H 4200 5150 50  0000 C CNN
 F 1 "10K" H 4200 5250 50  0000 C CNN
-F 2 "Resistors_SMD:R_0603" H 4050 5150 50  0001 C CNN
+F 2 "Resistors_SMD:R_0402" H 4050 5150 50  0001 C CNN
 F 3 "" H 4050 5150 50  0000 C CNN
 	1    4050 5150
@@
 P 2700 6050
 F 0 "TH1" V 2800 6100 50  0000 C CNN
-F 1 "THERMISTOR" V 2600 6050 50  0000 C BNN
-F 2 "" H 2700 6050 50  0001 C CNN
+F 1 "NCP15XW153J03RC" V 2600 6050 50  0000 C BNN
+F 2 "Resistors_SMD:R_0402" H 2700 6050 50  0001 C CNN
 F 3 "" H 2700 6050 50  0000 C CNN
 	1    2700 6050
@@
 F 0 "J10" H 1478 6241 50  0000 L CNN
 F 1 "CONN_01X02" H 1478 6150 50  0000 L CNN
-F 2 "sictroller:Molex-SL-2POS-RA" H 1400 6200 50  0001 C CNN
+F 2 "Connectors_Molex:Molex_PicoBlade_53261-0271" H 1400 6200 50  0001 C CNN
 F 3 "" H 1400 6200 50  0000 C CNN
 	1    1400 6200
@@
 F 0 "C55" H 6100 5550 50  0000 L CNN
 F 1 "0.1uF" H 6100 5450 50  0000 L CNN
-F 2 "Capacitors_SMD:C_0603" H 6000 5550 50  0001 C CNN
+F 2 "Capacitors_SMD:C_0402" H 6000 5550 50  0001 C CNN
 F 3 "" H 6000 5550 50  0000 C CNN
 	1    6000 5550
@@
 F 0 "R41" H 6150 5250 50  0000 C CNN
 F 1 "10K" H 6150 5350 50  0000 C CNN
-F 2 "Resistors_SMD:R_0603" H 6000 5250 50  0001 C CNN
+F 2 "Resistors_SMD:R_0402" H 6000 5250 50  0001 C CNN
 F 3 "" H 6000 5250 50  0000 C CNN
 	1    6000 5250
@@
 F 0 "Q1" H 6200 6150 50  0000 R CNN
 F 1 "CSD17483F4" H 6550 6050 50  0000 R CNN
-F 2 "" H 6100 6200 50  0001 C CNN
+F 2 "sictroller:FEMTOFET_YJC_YJJ" H 6100 6200 50  0001 C CNN
 F 3 "" H 5900 6100 50  0000 C CNN
 	1    5900 6100
@@
 F 0 "R43" H 6850 5500 50  0000 C CNN
 F 1 "56K" H 6850 5600 50  0000 C CNN
-F 2 "Resistors_SMD:R_0603" H 6700 5500 50  0001 C CNN
+F 2 "Resistors_SMD:R_0402" H 6700 5500 50  0001 C CNN
 F 3 "" H 6700 5500 50  0000 C CNN
 	1    6700 5500
@@
 F 0 "R45" H 6850 5800 50  0000 C CNN
 F 1 "100K" H 6850 5900 50  0000 C CNN
-F 2 "Resistors_SMD:R_0603" H 6700 5800 50  0001 C CNN
+F 2 "Resistors_SMD:R_0402" H 6700 5800 50  0001 C CNN
 F 3 "" H 6700 5800 50  0000 C CNN
 	1    6700 5800
@@
 F 0 "J8" H 7950 6050 50  0000 C CNN
 F 1 "RINGTERM" V 8050 5950 50  0000 C CNN
-F 2 "" H 7950 5950 50  0001 C CNN
+F 2 "sictroller:B6A-PCB" H 7950 5950 50  0001 C CNN
 F 3 "" H 7950 5950 50  0000 C CNN
 	1    7950 5950
@@
 F 0 "J9" H 9200 6050 50  0000 C CNN
 F 1 "RINGTERM" V 9300 5950 50  0000 C CNN
-F 2 "" H 9200 5950 50  0001 C CNN
+F 2 "sictroller:B6A-PCB" H 9200 5950 50  0001 C CNN
 F 3 "" H 9200 5950 50  0000 C CNN
 	1    9200 5950
@@
 	8350 6450 8350 6350
 Connection ~ 8350 6350
-Text Notes 7750 850  0    60   ~ 0
-Also, main high power external\nconnections are here.
+Text Notes 7750 800  0    60   ~ 0
+Also, main high power external connections are here.
 $Comp
 L C_Small C54
@@
 F 0 "C54" H 6300 5050 50  0000 L CNN
 F 1 "0.1uF" H 6300 4950 50  0000 L CNN
-F 2 "Capacitors_SMD:C_0603" H 6200 5050 50  0001 C CNN
+F 2 "Capacitors_SMD:C_0402" H 6200 5050 50  0001 C CNN
 F 3 "" H 6200 5050 50  0000 C CNN
 	1    6200 5050

Commit message: Footprint assignment complete
Parts:
- D7: footprint (none) -> Diodes_SMD:SOD-523
Changed lines of the file:
@@
 F 0 "D7" H 4300 5530 50  0000 L CNN
 F 1 "D_Schottky_Small" H 4070 5370 50  0000 L CNN
-F 2 "" V 4350 5450 50  0001 C CNN
+F 2 "Diodes_SMD:SOD-523" V 4350 5450 50  0001 C CNN
 F 3 "" V 4350 5450 50  0000 C CNN
 	1    4350 5450
