File: feedback.sch (KiCad schematic (older format))
At the start: 59 parts, among them J10 CONN_01X02, J11 RINGTERM, J12 RINGTERM, J4 RINGTERM, J5 RINGTERM, J6 RINGTERM, J7 CONN_01X02, J8 RINGTERM, J9 RINGTERM, Q1 CSD17483F4, U8 ADUM5241, U9 MAX6691

Commit message: Placed SiC module, DC link caps, HV / phase terminals
Connections:
- net A: now reaches I1.5 (IP-), J4.1 (P1)
- net B: now reaches I2.4 (IP+), J5.1 (P1)
- net C: now reaches I3.4 (IP+), J6.1 (P1)
Other:
- moved on the sheet: J4, J5, J6

Commit message: Add more ceralinks on rear
Parts:
- added TH2: NCP15XW153J03RC, Resistors_SMD:R_0402, symbol THERMISTOR
- added W23, W24: TEST_1P, Measurement_Points:Measurement_Point_Round-TH_Small, symbol TEST_1P
- renumbered C39 to C40, C40 to C41, C41 to C42, C42 to C43, C43 to C44, C44 to C45, C45 to C46, C46 to C47, C47 to C48, C48 to C49, C49 to C50, C50 to C51, C51 to C52, C52 to C53, C53 to C54, C54 to C55, C55 to C56, C56 to C57, R24 to R26, R25 to R27, R26 to R28, R27 to R29, R28 to R30, R29 to R31, R30 to R32, R31 to R33, R32 to R34, R33 to R35, R34 to R36, R35 to R37, R36 to R38, R37 to R39, R38 to R40, R39 to R41, R40 to R42, R41 to R43, R42 to R44, R43 to R45, R44 to R46, R45 to R47, R46 to R48
Connections:
- net CCS_NTC_2: now also W24.1; no longer TH1.2
- net at U9.4 (T4): now also W23.1; no longer TH1.1
- new net: TH1.1, TH2.1
- new net: TH1.2, TH2.2
Other:
- note added: "Externally wired"
- moved on the sheet: TH1

Commit message: Improved footprint for B6A-PCB
Parts:
- TH1, TH2: footprint Resistors_SMD:R_0402 -> sictroller:R_0402_extwire
Connections:
- net A: now also I1.4 (IP+); no longer I1.5 (IP-)
- net B: now also I2.5 (IP-); no longer I2.4 (IP+)
- net C: now also I3.5 (IP-); no longer I3.4 (IP+)
- net PHASE_A: now also I1.5 (IP-); no longer I1.4 (IP+)
- net PHASE_B: now also I2.4 (IP+); no longer I2.5 (IP-)
- net PHASE_C: now also I3.4 (IP+); no longer I3.5 (IP-)
- net at TH1.1: no longer TH2.1
- net at TH1.2: no longer TH2.2
- no-connect marks 0 -> 4
Other:
- moved on the sheet: J4, J5, J6
Changed lines of the file:
@@
 	1    0    0    -1
 $EndComp
-Text GLabel 8300 3400 0    60   UnSpc ~ 0
+Text GLabel 8300 2900 0    60   UnSpc ~ 0
 PHASE_B
-Text GLabel 8300 5200 0    60   UnSpc ~ 0
+Text GLabel 8300 4700 0    60   UnSpc ~ 0
 PHASE_C
-Text GLabel 8300 1100 0    60   UnSpc ~ 0
+Text GLabel 8300 1600 0    60   UnSpc ~ 0
 PHASE_A
 $Comp
 L CONN_01X01 J4
 U 1 1 57F392C3
-P 7950 1600
-F 0 "J4" H 7950 1700 50  0000 C CNN
-F 1 "RINGTERM" V 8050 1600 50  0000 C CNN
-F 2 "sictroller:B6A-PCB" H 7950 1600 50  0001 C CNN
-F 3 "" H 7950 1600 50  0000 C CNN
-	1    7950 1600
+P 8100 1100
+F 0 "J4" H 8100 1200 50  0000 C CNN
+F 1 "RINGTERM" V 8200 1100 50  0000 C CNN
+F 2 "sictroller:B6A-PCB" H 8100 1100 50  0001 C CNN
+F 3 "" H 8100 1100 50  0000 C CNN
+	1    8100 1100
 	-1   0    0    1
 $EndComp
@@
 L CONN_01X01 J5
 U 1 1 57F39459
-P 7950 2900
-F 0 "J5" H 7950 3000 50  0000 C CNN
-F 1 "RINGTERM" V 8050 2900 50  0000 C CNN
-F 2 "sictroller:B6A-PCB" H 7950 2900 50  0001 C CNN
-F 3 "" H 7950 2900 50  0000 C CNN
-	1    7950 2900
+P 8100 3400
+F 0 "J5" H 8100 3500 50  0000 C CNN
+F 1 "RINGTERM" V 8200 3400 50  0000 C CNN
+F 2 "sictroller:B6A-PCB" H 8100 3400 50  0001 C CNN
+F 3 "" H 8100 3400 50  0000 C CNN
+	1    8100 3400
 	-1   0    0    1
 $EndComp
@@
 L CONN_01X01 J6
 U 1 1 57F39531
-P 7950 4700
-F 0 "J6" H 7950 4800 50  0000 C CNN
-F 1 "RINGTERM" V 8050 4700 50  0000 C CNN
-F 2 "sictroller:B6A-PCB" H 7950 4700 50  0001 C CNN
-F 3 "" H 7950 4700 50  0000 C CNN
-	1    7950 4700
+P 8100 5200
+F 0 "J6" H 8100 5300 50  0000 C CNN
+F 1 "RINGTERM" V 8200 5200 50  0000 C CNN
+F 2 "sictroller:B6A-PCB" H 8100 5200 50  0001 C CNN
+F 3 "" H 8100 5200 50  0000 C CNN
+	1    8100 5200
 	-1   0    0    1
 $EndComp
@@
 F 0 "TH1" V 3150 6700 50  0000 C CNN
 F 1 "NCP15XW153J03RC" V 2950 6650 50  0000 C BNN
-F 2 "Resistors_SMD:R_0402" H 3050 6650 50  0001 C CNN
+F 2 "sictroller:R_0402_extwire" H 3050 6650 50  0001 C CNN
 F 3 "" H 3050 6650 50  0000 C CNN
 	1    3050 6650
@@
 	2400 6300 2400 5350
 Connection ~ 2400 5350
-Wire Wire Line
-	8150 1600 8300 1600
-Text Label 8150 1600 0    60   ~ 0
+Text Label 8300 1100 0    60   ~ 0
 A
-Wire Wire Line
-	8150 2900 8300 2900
-Text Label 8150 2900 0    60   ~ 0
+Text Label 8300 3400 0    60   ~ 0
 B
-Wire Wire Line
-	8150 4700 8300 4700
-Text Label 8150 4700 0    60   ~ 0
+Text Label 8300 5200 0    60   ~ 0
 C
 Text Notes 2650 7100 0    60   ~ 0
@@
 F 0 "TH2" V 3150 6950 50  0000 C CNN
 F 1 "NCP15XW153J03RC" V 2950 6900 50  0000 C BNN
-F 2 "Resistors_SMD:R_0402" H 3050 6900 50  0001 C CNN
+F 2 "sictroller:R_0402_extwire" H 3050 6900 50  0001 C CNN
 F 3 "" H 3050 6900 50  0000 C CNN
 	1    3050 6900
 	0    1    1    0
 $EndComp
-Wire Wire Line
-	2800 6650 2800 6900
-Wire Wire Line
-	3300 6650 3300 6900
+NoConn ~ 3300 6650
+NoConn ~ 3300 6900
+NoConn ~ 2800 6900
+NoConn ~ 2800 6650
 $EndSCHEMATC

Commit message: some logic placement progress
Connections:
- net GNDD: no longer C40.2, C41.2, C42.2, C43.2, C44.2, C45.2, C46.2, C47.2, C48.2, C49.2, C50.2, C51.2, C54.2, C57.2, I1.2 (GND), I2.2 (GND), I3.2 (GND), R31.1, R36.1, R37.1, R38.1, R39.1, R41.1, R46.1
- new net GNDA: C40.2, C41.2, C42.2, C43.2, C44.2, C45.2, C46.2, C47.2, C48.2, C49.2, C50.2, C51.2, C54.2, C57.2, I1.2 (GND), I2.2 (GND), I3.2 (GND), R31.1, R36.1, R37.1, R38.1, R39.1, R41.1, R46.1
Changed lines of the file:
@@
 Todo: Vphase peak detection
-$Comp
-L GNDD #PWR071
-U 1 1 57A42A2E
-P 2250 2650
-F 0 "#PWR071" H 2250 2400 50  0001 C CNN
-F 1 "GNDD" H 2250 2500 50  0000 C CNN
-F 2 "" H 2250 2650 50  0000 C CNN
-F 3 "" H 2250 2650 50  0000 C CNN
-	1    2250 2650
-	-1   0    0    -1
-$EndComp
 $Comp
 L R_Small R28
@@
 $EndComp
 $Comp
-L GNDD #PWR072
-U 1 1 57A43050
-P 3150 2650
-F 0 "#PWR072" H 3150 2400 50  0001 C CNN
-F 1 "GNDD" H 3150 2500 50  0000 C CNN
-F 2 "" H 3150 2650 50  0000 C CNN
-F 3 "" H 3150 2650 50  0000 C CNN
-	1    3150 2650
-	-1   0    0    -1
-$EndComp
-$Comp
 L R_Small R29
 U 1 1 57A4320A
@@
 $EndComp
 $Comp
-L GNDD #PWR073
-U 1 1 57A43227
-P 4100 2650
-F 0 "#PWR073" H 4100 2400 50  0001 C CNN
-F 1 "GNDD" H 4100 2500 50  0000 C CNN
-F 2 "" H 4100 2650 50  0000 C CNN
-F 3 "" H 4100 2650 50  0000 C CNN
-	1    4100 2650
-	-1   0    0    -1
-$EndComp
-$Comp
 L R_Small R30
 U 1 1 57A4322F
@@
 $EndComp
 $Comp
-L GNDD #PWR074
-U 1 1 57A4324C
-P 5050 2650
-F 0 "#PWR074" H 5050 2400 50  0001 C CNN
-F 1 "GNDD" H 5050 2500 50  0000 C CNN
-F 2 "" H 5050 2650 50  0000 C CNN
-F 3 "" H 5050 2650 50  0000 C CNN
-	1    5050 2650
-	-1   0    0    -1
-$EndComp
-$Comp
 L +5VA #PWR075
 U 1 1 57A45500
@@
 $EndComp
 $Comp
-L GNDD #PWR076
-U 1 1 57A455E4
-P 9500 1350
-F 0 "#PWR076" H 9500 1100 50  0001 C CNN
-F 1 "GNDD" H 9500 1200 50  0000 C CNN
-F 2 "" H 9500 1350 50  0000 C CNN
-F 3 "" H 9500 1350 50  0000 C CNN
-	1    9500 1350
-	-1   0    0    -1
-$EndComp
-$Comp
 L R_Small R26
 U 1 1 57A45AEC
@@
 $EndComp
 $Comp
-L GNDD #PWR077
-U 1 1 57A45B03
-P 9800 2250
-F 0 "#PWR077" H 9800 2000 50  0001 C CNN
-F 1 "GNDD" H 9800 2100 50  0000 C CNN
-F 2 "" H 9800 2250 50  0000 C CNN
-F 3 "" H 9800 2250 50  0000 C CNN
-	1    9800 2250
-	-1   0    0    -1
-$EndComp
-$Comp
-L +5VA #PWR078
+L +5VA #PWR076
 U 1 1 57A475BB
 P 9500 2850
-F 0 "#PWR078" H 9500 2700 50  0001 C CNN
+F 0 "#PWR076" H 9500 2700 50  0001 C CNN
 F 1 "+5VA" H 9515 3023 50  0000 C CNN
 F 2 "" H 9500 2850 50  0000 C CNN
@@
 $EndComp
 $Comp
-L GNDD #PWR079
-U 1 1 57A475DE
-P 9800 4050
-F 0 "#PWR079" H 9800 3800 50  0001 C CNN
-F 1 "GNDD" H 9800 3900 50  0000 C CNN
-F 2 "" H 9800 4050 50  0000 C CNN
-F 3 "" H 9800 4050 50  0000 C CNN
-	1    9800 4050
-	-1   0    0    -1
-$EndComp
-$Comp
-L +5VA #PWR080
+L +5VA #PWR077
 U 1 1 57A47980
 P 9500 4650
-F 0 "#PWR080" H 9500 4500 50  0001 C CNN
+F 0 "#PWR077" H 9500 4500 50  0001 C CNN
 F 1 "+5VA" H 9515 4823 50  0000 C CNN
 F 2 "" H 9500 4650 50  0000 C CNN
@@
 	1    10000 5700
 	1    0    0    -1
-$EndComp
-$Comp
-L GNDD #PWR081
-U 1 1 57A479A3
-P 9800 5850
-F 0 "#PWR081" H 9800 5600 50  0001 C CNN
-F 1 "GNDD" H 9800 5700 50  0000 C CNN
-F 2 "" H 9800 5850 50  0000 C CNN
-F 3 "" H 9800 5850 50  0000 C CNN
-	1    9800 5850
-	-1   0    0    -1
 $EndComp
 $Comp
@@
 BUS+
 $Comp
-L ACS770 I1
-U 1 1 57F3202F
-P 8900 1350
-F 0 "I1" H 8900 1200 60  0000 C CNN
-F 1 "ACS770" H 8900 1500 60  0000 C CNN
-F 2 "sictroller:ACS770" H 8900 1350 60  0001 C CNN
-F 3 "" H 8900 1350 60  0000 C CNN
-	1    8900 1350
-	1    0    0    -1
-$EndComp
-$Comp
 L ACS770 I2
 U 1 1 57F330A0
@@
 	1    8900 4950
 	1    0    0    -1
-$EndComp
-$Comp
-L GNDD #PWR082
-U 1 1 57F3436C
-P 9500 3150
-F 0 "#PWR082" H 9500 2900 50  0001 C CNN
-F 1 "GNDD" H 9500 3000 50  0000 C CNN
-F 2 "" H 9500 3150 50  0000 C CNN
-F 3 "" H 9500 3150 50  0000 C CNN
-	1    9500 3150
-	-1   0    0    -1
-$EndComp
-$Comp
-L GNDD #PWR083
-U 1 1 57F3441F
-P 9500 4950
-F 0 "#PWR083" H 9500 4700 50  0001 C CNN
-F 1 "GNDD" H 9500 4800 50  0000 C CNN
-F 2 "" H 9500 4950 50  0000 C CNN
-F 3 "" H 9500 4950 50  0000 C CNN
-	1    9500 4950
-	-1   0    0    -1
 $EndComp
 $Comp
@@
 $EndComp
 $Comp
-L +5VD #PWR084
+L +5VD #PWR078
 U 1 1 57F6CCA4
 P 5650 5150
-F 0 "#PWR084" H 5650 5000 50  0001 C CNN
+F 0 "#PWR078" H 5650 5000 50  0001 C CNN
 F 1 "+5VD" H 5650 5290 50  0000 C CNN
 F 2 "" H 5650 5150 50  0000 C CNN
@@
 $EndComp
 $Comp
-L GNDD #PWR085
+L GNDD #PWR079
 U 1 1 57F6AC00
 P 6000 6350
-F 0 "#PWR085" H 6000 6100 50  0001 C CNN
+F 0 "#PWR079" H 6000 6100 50  0001 C CNN
 F 1 "GNDD" H 6000 6200 50  0000 C CNN
 F 2 "" H 6000 6350 50  0000 C CNN
@@
 $EndComp
 $Comp
-L GNDD #PWR086
+L GNDD #PWR080
 U 1 1 57F6EE21
 P 6700 6050
-F 0 "#PWR086" H 6700 5800 50  0001 C CNN
+F 0 "#PWR080" H 6700 5800 50  0001 C CNN
 F 1 "GNDD" H 6700 5900 50  0000 C CNN
 F 2 "" H 6700 6050 50  0000 C CNN
@@
 $EndComp
 $Comp
-L GNDD #PWR087
+L GNDD #PWR081
 U 1 1 57FC3D16
 P 6200 5150
-F 0 "#PWR087" H 6200 4900 50  0001 C CNN
+F 0 "#PWR081" H 6200 4900 50  0001 C CNN
 F 1 "GNDD" H 6200 5000 50  0000 C CNN
 F 2 "" H 6200 5150 50  0000 C CNN
@@
 $EndComp
 $Comp
-L PWR_FLAG #FLG088
+L PWR_FLAG #FLG082
 U 1 1 57FCFCD0
 P 5700 5700
-F 0 "#FLG088" H 5700 5795 50  0001 C CNN
+F 0 "#FLG082" H 5700 5795 50  0001 C CNN
 F 1 "PWR_FLAG" H 5700 5880 50  0000 C CNN
 F 2 "" H 5700 5700 50  0000 C CNN
@@
 NoConn ~ 2800 6900
 NoConn ~ 2800 6650
+$Comp
+L GNDA #PWR083
+U 1 1 5806BCAA
+P 9800 2250
+F 0 "#PWR083" H 9800 2000 50  0001 C CNN
+F 1 "GNDA" H 9800 2100 50  0000 C CNN
+F 2 "" H 9800 2250 50  0000 C CNN
+F 3 "" H 9800 2250 50  0000 C CNN
+	1    9800 2250
+	1    0    0    -1
+$EndComp
+$Comp
+L GNDA #PWR084
+U 1 1 5806C298
+P 9800 4050
+F 0 "#PWR084" H 9800 3800 50  0001 C CNN
+F 1 "GNDA" H 9800 3900 50  0000 C CNN
+F 2 "" H 9800 4050 50  0000 C CNN
+F 3 "" H 9800 4050 50  0000 C CNN
+	1    9800 4050
+	1    0    0    -1
+$EndComp
+$Comp
+L GNDA #PWR085
+U 1 1 5806C35D
+P 9800 5850
+F 0 "#PWR085" H 9800 5600 50  0001 C CNN
+F 1 "GNDA" H 9800 5700 50  0000 C CNN
+F 2 "" H 9800 5850 50  0000 C CNN
+F 3 "" H 9800 5850 50  0000 C CNN
+	1    9800 5850
+	1    0    0    -1
+$EndComp
+$Comp
+L ACS770 I1
+U 1 1 57F3202F
+P 8900 1350
+F 0 "I1" H 8900 1200 60  0000 C CNN
+F 1 "ACS770" H 8900 1500 60  0000 C CNN
+F 2 "sictroller:ACS770" H 8900 1350 60  0001 C CNN
+F 3 "" H 8900 1350 60  0000 C CNN
+	1    8900 1350
+	1    0    0    -1
+$EndComp
+$Comp
+L GNDA #PWR086
+U 1 1 5806C55B
+P 9500 1350
+F 0 "#PWR086" H 9500 1100 50  0001 C CNN
+F 1 "GNDA" H 9500 1200 50  0000 C CNN
+F 2 "" H 9500 1350 50  0000 C CNN
+F 3 "" H 9500 1350 50  0000 C CNN
+	1    9500 1350
+	1    0    0    -1
+$EndComp
+$Comp
+L GNDA #PWR087
+U 1 1 5806C620
+P 9500 3150
+F 0 "#PWR087" H 9500 2900 50  0001 C CNN
+F 1 "GNDA" H 9500 3000 50  0000 C CNN
+F 2 "" H 9500 3150 50  0000 C CNN
+F 3 "" H 9500 3150 50  0000 C CNN
+	1    9500 3150
+	1    0    0    -1
+$EndComp
+$Comp
+L GNDA #PWR088
+U 1 1 5806C6E5
+P 9500 4950
+F 0 "#PWR088" H 9500 4700 50  0001 C CNN
+F 1 "GNDA" H 9500 4800 50  0000 C CNN
+F 2 "" H 9500 4950 50  0000 C CNN
+F 3 "" H 9500 4950 50  0000 C CNN
+	1    9500 4950
+	1    0    0    -1
+$EndComp
+$Comp
+L GNDA #PWR089
+U 1 1 5806D1DA
+P 5050 2650
+F 0 "#PWR089" H 5050 2400 50  0001 C CNN
+F 1 "GNDA" H 5050 2500 50  0000 C CNN
+F 2 "" H 5050 2650 50  0000 C CNN
+F 3 "" H 5050 2650 50  0000 C CNN
+	1    5050 2650
+	1    0    0    -1
+$EndComp
+$Comp
+L GNDA #PWR090
+U 1 1 5806D451
+P 4100 2650
+F 0 "#PWR090" H 4100 2400 50  0001 C CNN
+F 1 "GNDA" H 4100 2500 50  0000 C CNN
+F 2 "" H 4100 2650 50  0000 C CNN
+F 3 "" H 4100 2650 50  0000 C CNN
+	1    4100 2650
+	1    0    0    -1
+$EndComp
+$Comp
+L GNDA #PWR091
+U 1 1 5806D516
+P 3150 2650
+F 0 "#PWR091" H 3150 2400 50  0001 C CNN
+F 1 "GNDA" H 3150 2500 50  0000 C CNN
+F 2 "" H 3150 2650 50  0000 C CNN
+F 3 "" H 3150 2650 50  0000 C CNN
+	1    3150 2650
+	1    0    0    -1
+$EndComp
+$Comp
+L GNDA #PWR092
+U 1 1 5806D5DB
+P 2250 2650
+F 0 "#PWR092" H 2250 2400 50  0001 C CNN
+F 1 "GNDA" H 2250 2500 50  0000 C CNN
+F 2 "" H 2250 2650 50  0000 C CNN
+F 3 "" H 2250 2650 50  0000 C CNN
+	1    2250 2650
+	1    0    0    -1
+$EndComp
 $EndSCHEMATC

Commit message: Placement almost complete
Parts:
- C43, C45, C47, C49: footprint Capacitors_SMD:C_0603 -> Capacitors_SMD:C_0402
- C48: value 100 nF C0G 1% -> 0.1uF 10V; footprint Capacitors_SMD:C_1210 -> Capacitors_SMD:C_0402
- R36, R37, R38, R39: footprint Resistors_SMD:R_0603 -> Resistors_SMD:R_0402
Other:
- note removed: "Place C28/29/30/31\nnear signal entrance"
Changed lines of the file:
@@
 F 0 "R36" H 2400 2500 50  0000 C CNN
 F 1 "3.6K 1%" V 2145 2500 50  0001 C CNN
-F 2 "Resistors_SMD:R_0603" H 2250 2500 50  0001 C CNN
+F 2 "Resistors_SMD:R_0402" H 2250 2500 50  0001 C CNN
 F 3 "" H 2250 2500 50  0000 C CNN
 	1    2250 2500
@@
 F 0 "R37" H 3300 2500 50  0000 C CNN
 F 1 "3.6K 1%" V 3045 2500 50  0001 C CNN
-F 2 "Resistors_SMD:R_0603" H 3150 2500 50  0001 C CNN
+F 2 "Resistors_SMD:R_0402" H 3150 2500 50  0001 C CNN
 F 3 "" H 3150 2500 50  0000 C CNN
 	1    3150 2500
@@
 P 4100 2500
 F 0 "R38" H 4250 2500 50  0000 C CNN
-F 1 "3.6K 1%" V 3995 2500 50  0001 C CNN
-F 2 "Resistors_SMD:R_0603" H 4100 2500 50  0001 C CNN
+F 1 "3.6K 1%" V 4100 3150 50  0000 C CNN
+F 2 "Resistors_SMD:R_0402" H 4100 2500 50  0001 C CNN
 F 3 "" H 4100 2500 50  0000 C CNN
 	1    4100 2500
@@
 P 4300 2500
 F 0 "C46" H 4200 2350 50  0000 L CNN
-F 1 "100 nF C0G 1%" H 4392 2455 50  0001 L CNN
+F 1 "100 nF C0G 1%" V 4300 1600 50  0000 L CNN
 F 2 "Capacitors_SMD:C_1210" H 4300 2500 50  0001 C CNN
 F 3 "" H 4300 2500 50  0000 C CNN
@@
 F 0 "R39" H 5200 2500 50  0000 C CNN
 F 1 "3.6K 1%" V 5050 3150 50  0000 C CNN
-F 2 "Resistors_SMD:R_0603" H 5050 2500 50  0001 C CNN
+F 2 "Resistors_SMD:R_0402" H 5050 2500 50  0001 C CNN
 F 3 "" H 5050 2500 50  0000 C CNN
 	1    5050 2500
@@
 P 5250 2500
 F 0 "C48" H 5150 2350 50  0000 L CNN
-F 1 "100 nF C0G 1%" V 5250 1650 50  0000 L CNN
-F 2 "Capacitors_SMD:C_1210" H 5250 2500 50  0001 C CNN
+F 1 "0.1uF 10V" V 5250 1650 50  0000 L CNN
+F 2 "Capacitors_SMD:C_0402" H 5250 2500 50  0001 C CNN
 F 3 "" H 5250 2500 50  0000 C CNN
 	1    5250 2500
@@
 F 0 "C49" H 5492 2546 50  0000 L CNN
 F 1 "470pF" V 5400 1800 50  0000 L CNN
-F 2 "Capacitors_SMD:C_0603" H 5400 2500 50  0001 C CNN
+F 2 "Capacitors_SMD:C_0402" H 5400 2500 50  0001 C CNN
 F 3 "" H 5400 2500 50  0000 C CNN
 	1    5400 2500
@@
 F 0 "C43" H 2692 2500 50  0000 L CNN
 F 1 "470pF" H 2692 2455 50  0001 L CNN
-F 2 "Capacitors_SMD:C_0603" H 2600 2500 50  0001 C CNN
+F 2 "Capacitors_SMD:C_0402" H 2600 2500 50  0001 C CNN
 F 3 "" H 2600 2500 50  0000 C CNN
 	1    2600 2500
@@
 F 0 "C45" H 3592 2500 50  0000 L CNN
 F 1 "470pF" H 3592 2455 50  0001 L CNN
-F 2 "Capacitors_SMD:C_0603" H 3500 2500 50  0001 C CNN
+F 2 "Capacitors_SMD:C_0402" H 3500 2500 50  0001 C CNN
 F 3 "" H 3500 2500 50  0000 C CNN
 	1    3500 2500
@@
 P 4450 2500
 F 0 "C47" H 4542 2500 50  0000 L CNN
-F 1 "470pF" H 4542 2455 50  0001 L CNN
-F 2 "Capacitors_SMD:C_0603" H 4450 2500 50  0001 C CNN
+F 1 "470pF" V 4450 1750 50  0000 L CNN
+F 2 "Capacitors_SMD:C_0402" H 4450 2500 50  0001 C CNN
 F 3 "" H 4450 2500 50  0000 C CNN
 	1    4450 2500
 	1    0    0    -1
 $EndComp
-Text Notes 5450 2850 0    43   ~ 0
-Place C28/29/30/31\nnear signal entrance
 Text GLabel 1550 1400 0    60   UnSpc ~ 0
 PHASE_C
