File: powerstage-CCS050M12CM2.sch (KiCad schematic (older format))
At the start: 34 parts, among them J13 CONN_01X01, Q2 CCS050M12CM2, U10 74LVC2G04, U11 74LVC8T245

Commit message: Footprints assigned for all except halfbridge-driver
Parts:
- removed U11: 74LVC8T245, Housings_SSOP:TSSOP-24_4.4x7.8mm_Pitch0.65mm, symbol 74LVC8T245
- added U11: TXS0108E, sictroller:VQFN-20, symbol TXS0108E
- C57, C58, C59: footprint Capacitors_SMD:C_0603 -> Capacitors_SMD:C_0402
- C62, C63, C64, C65, C66, C67, C68, C69, C70, C71, C72, C73, C74, C75, C76, C77: footprint Capacitors_SMD:C_0603 -> sictroller:Ceralink-L
- J13: footprint (none) -> Measurement_Points:Measurement_Point_Round-TH_Small
- Q2: footprint (none) -> sictroller:6pack-45mm
- R47, R48, R49, R50, R51, R52, R53: footprint Resistors_SMD:R_0603 -> Resistors_SMD:R_0402
Connections:
- net +3V3: now also U11.10 (OE), U11.2 (VccA), U11.9 (A8)
- net +5VD: now also U11.19 (VccB)
- net GND: now also U11.11 (GND), U11.PAD (GND)
- net PWM_AH: now also U11.8 (A7)
- net PWM_AH_TTL: now also U11.13 (B7)
- net PWM_AL: now also U11.7 (A6)
- net PWM_AL_TTL: now also U11.14 (B6)
- net PWM_BH: now also U11.6 (A5)
- net PWM_BH_TTL: now also U11.15 (B5)
- net PWM_BL: now also U11.5 (A4)
- net PWM_BL_TTL: now also U11.16 (B4)
- net PWM_CH: now also U11.4 (A3)
- net PWM_CH_TTL: now also U11.17 (B3)
- net PWM_CL: now also U11.3 (A2)
- net PWM_CL_TTL: now also U11.18 (B2)
- net ~PWR_RESET: now also U11.1 (A1)
- net ~PWR_RESET_TTL: now also U11.20 (B1)
Other:
- note added: "TODO: Softer level shifter?"
Changed lines of the file:
@@
 $EndDescr
-$Comp
-L 74LVC8T245 U11
-U 1 1 57A19094
-P 3650 5350
-F 0 "U11" H 3450 6300 60  0000 L CNN
-F 1 "74LVC8T245" H 3450 4500 60  0000 L CNN
-F 2 "Housings_SSOP:TSSOP-24_4.4x7.8mm_Pitch0.65mm" H 3650 4650 60  0001 C CNN
-F 3 "" H 3650 4650 60  0000 C CNN
-	1    3650 5350
-	1    0    0    -1
-$EndComp
 $Comp
 L +5VD #PWR086
@@
 F 0 "R47" H 2630 4670 50  0000 L CNN
 F 1 "10k" H 2630 4610 50  0000 L CNN
-F 2 "Resistors_SMD:R_0603" H 2600 4650 50  0001 C CNN
+F 2 "Resistors_SMD:R_0402" H 2600 4650 50  0001 C CNN
 F 3 "" H 2600 4650 50  0000 C CNN
 	1    2600 4650
@@
 F 0 "C59" H 4310 4520 50  0000 L CNN
 F 1 "0.1uF" H 4310 4370 50  0000 L CNN
-F 2 "Capacitors_SMD:C_0603" H 4300 4450 50  0001 C CNN
+F 2 "Capacitors_SMD:C_0402" H 4300 4450 50  0001 C CNN
 F 3 "" H 4300 4450 50  0000 C CNN
 	1    4300 4450
@@
 L GNDD #PWR090
 U 1 1 57A19193
-P 3250 6300
-F 0 "#PWR090" H 3250 6050 50  0001 C CNN
-F 1 "GNDD" H 3250 6150 50  0000 C CNN
-F 2 "" H 3250 6300 50  0000 C CNN
-F 3 "" H 3250 6300 50  0000 C CNN
-	1    3250 6300
+P 3250 5950
+F 0 "#PWR090" H 3250 5700 50  0001 C CNN
+F 1 "GNDD" H 3250 5800 50  0000 C CNN
+F 2 "" H 3250 5950 50  0000 C CNN
+F 3 "" H 3250 5950 50  0000 C CNN
+	1    3250 5950
 	1    0    0    -1
 $EndComp
@@
 F 0 "C58" H 2960 4520 50  0000 L CNN
 F 1 "0.1uF" H 2960 4370 50  0000 L CNN
-F 2 "Capacitors_SMD:C_0603" H 2950 4450 50  0001 C CNN
+F 2 "Capacitors_SMD:C_0402" H 2950 4450 50  0001 C CNN
 F 3 "" H 2950 4450 50  0000 C CNN
 	1    2950 4450
@@
 F 0 "C57" H 2510 1420 50  0000 L CNN
 F 1 "0.1uF" H 2510 1270 50  0000 L CNN
-F 2 "Capacitors_SMD:C_0603" H 2500 1350 50  0001 C CNN
+F 2 "Capacitors_SMD:C_0402" H 2500 1350 50  0001 C CNN
 F 3 "" H 2500 1350 50  0000 C CNN
 	1    2500 1350
@@
 F 0 "Q2" H 8550 4400 60  0000 L CNN
 F 1 "CCS050M12CM2" H 9750 4400 60  0000 R CNN
-F 2 "" H 9150 2750 60  0001 C CNN
+F 2 "sictroller:6pack-45mm" H 9150 2750 60  0001 C CNN
 F 3 "" H 9150 2750 60  0000 C CNN
 	1    9150 3450
@@
 F 0 "R48" H 1430 5770 50  0000 L CNN
 F 1 "10k" H 1430 5710 50  0000 L CNN
-F 2 "Resistors_SMD:R_0603" H 1400 5750 50  0001 C CNN
+F 2 "Resistors_SMD:R_0402" H 1400 5750 50  0001 C CNN
 F 3 "" H 1400 5750 50  0000 C CNN
 	1    1400 5750
@@
 F 0 "R49" H 1730 5770 50  0000 L CNN
 F 1 "10k" H 1730 5710 50  0000 L CNN
-F 2 "Resistors_SMD:R_0603" H 1700 5750 50  0001 C CNN
+F 2 "Resistors_SMD:R_0402" H 1700 5750 50  0001 C CNN
 F 3 "" H 1700 5750 50  0000 C CNN
 	1    1700 5750
@@
 F 0 "R50" H 2030 5770 50  0000 L CNN
 F 1 "10k" H 2030 5710 50  0000 L CNN
-F 2 "Resistors_SMD:R_0603" H 2000 5750 50  0001 C CNN
+F 2 "Resistors_SMD:R_0402" H 2000 5750 50  0001 C CNN
 F 3 "" H 2000 5750 50  0000 C CNN
 	1    2000 5750
@@
 F 0 "R51" H 2330 5770 50  0000 L CNN
 F 1 "10k" H 2330 5710 50  0000 L CNN
-F 2 "Resistors_SMD:R_0603" H 2300 5750 50  0001 C CNN
+F 2 "Resistors_SMD:R_0402" H 2300 5750 50  0001 C CNN
 F 3 "" H 2300 5750 50  0000 C CNN
 	1    2300 5750
@@
 F 0 "R52" H 2630 5770 50  0000 L CNN
 F 1 "10k" H 2630 5710 50  0000 L CNN
-F 2 "Resistors_SMD:R_0603" H 2600 5750 50  0001 C CNN
+F 2 "Resistors_SMD:R_0402" H 2600 5750 50  0001 C CNN
 F 3 "" H 2600 5750 50  0000 C CNN
 	1    2600 5750
@@
 F 0 "R53" H 2930 5770 50  0000 L CNN
 F 1 "10k" H 2930 5710 50  0000 L CNN
-F 2 "Resistors_SMD:R_0603" H 2900 5750 50  0001 C CNN
+F 2 "Resistors_SMD:R_0402" H 2900 5750 50  0001 C CNN
 F 3 "" H 2900 5750 50  0000 C CNN
 	1    2900 5750
@@
 F 0 "C62" H 1310 7220 50  0000 L CNN
 F 1 "1uF" H 1310 7070 50  0000 L CNN
-F 2 "Capacitors_SMD:C_0603" H 1300 7150 50  0001 C CNN
+F 2 "sictroller:Ceralink-L" H 1300 7150 50  0001 C CNN
 F 3 "" H 1300 7150 50  0000 C CNN
 	1    1300 7150
@@
 F 0 "C63" H 1510 7220 50  0000 L CNN
 F 1 "1uF" H 1510 7070 50  0000 L CNN
-F 2 "Capacitors_SMD:C_0603" H 1500 7150 50  0001 C CNN
+F 2 "sictroller:Ceralink-L" H 1500 7150 50  0001 C CNN
 F 3 "" H 1500 7150 50  0000 C CNN
 	1    1500 7150
@@
 F 0 "C64" H 1710 7220 50  0000 L CNN
 F 1 "1uF" H 1710 7070 50  0000 L CNN
-F 2 "Capacitors_SMD:C_0603" H 1700 7150 50  0001 C CNN
+F 2 "sictroller:Ceralink-L" H 1700 7150 50  0001 C CNN
 F 3 "" H 1700 7150 50  0000 C CNN
 	1    1700 7150
@@
 F 0 "C65" H 1910 7220 50  0000 L CNN
 F 1 "1uF" H 1910 7070 50  0000 L CNN
-F 2 "Capacitors_SMD:C_0603" H 1900 7150 50  0001 C CNN
+F 2 "sictroller:Ceralink-L" H 1900 7150 50  0001 C CNN
 F 3 "" H 1900 7150 50  0000 C CNN
 	1    1900 7150
@@
 F 0 "C66" H 2110 7220 50  0000 L CNN
 F 1 "1uF" H 2110 7070 50  0000 L CNN
-F 2 "Capacitors_SMD:C_0603" H 2100 7150 50  0001 C CNN
+F 2 "sictroller:Ceralink-L" H 2100 7150 50  0001 C CNN
 F 3 "" H 2100 7150 50  0000 C CNN
 	1    2100 7150
@@
 F 0 "C67" H 2310 7220 50  0000 L CNN
 F 1 "1uF" H 2310 7070 50  0000 L CNN
-F 2 "Capacitors_SMD:C_0603" H 2300 7150 50  0001 C CNN
+F 2 "sictroller:Ceralink-L" H 2300 7150 50  0001 C CNN
 F 3 "" H 2300 7150 50  0000 C CNN
 	1    2300 7150
@@
 F 0 "C68" H 2510 7220 50  0000 L CNN
 F 1 "1uF" H 2510 7070 50  0000 L CNN
-F 2 "Capacitors_SMD:C_0603" H 2500 7150 50  0001 C CNN
+F 2 "sictroller:Ceralink-L" H 2500 7150 50  0001 C CNN
 F 3 "" H 2500 7150 50  0000 C CNN
 	1    2500 7150
@@
 F 0 "C69" H 2710 7220 50  0000 L CNN
 F 1 "1uF" H 2710 7070 50  0000 L CNN
-F 2 "Capacitors_SMD:C_0603" H 2700 7150 50  0001 C CNN
+F 2 "sictroller:Ceralink-L" H 2700 7150 50  0001 C CNN
 F 3 "" H 2700 7150 50  0000 C CNN
 	1    2700 7150
@@
 F 0 "C70" H 2910 7220 50  0000 L CNN
 F 1 "1uF" H 2910 7070 50  0000 L CNN
-F 2 "Capacitors_SMD:C_0603" H 2900 7150 50  0001 C CNN
+F 2 "sictroller:Ceralink-L" H 2900 7150 50  0001 C CNN
 F 3 "" H 2900 7150 50  0000 C CNN
 	1    2900 7150
@@
 F 0 "C71" H 3110 7220 50  0000 L CNN
 F 1 "1uF" H 3110 7070 50  0000 L CNN
-F 2 "Capacitors_SMD:C_0603" H 3100 7150 50  0001 C CNN
+F 2 "sictroller:Ceralink-L" H 3100 7150 50  0001 C CNN
 F 3 "" H 3100 7150 50  0000 C CNN
 	1    3100 7150
@@
 F 0 "C72" H 3310 7220 50  0000 L CNN
 F 1 "1uF" H 3310 7070 50  0000 L CNN
-F 2 "Capacitors_SMD:C_0603" H 3300 7150 50  0001 C CNN
+F 2 "sictroller:Ceralink-L" H 3300 7150 50  0001 C CNN
 F 3 "" H 3300 7150 50  0000 C CNN
 	1    3300 7150
@@
 F 0 "C73" H 3510 7220 50  0000 L CNN
 F 1 "1uF" H 3510 7070 50  0000 L CNN
-F 2 "Capacitors_SMD:C_0603" H 3500 7150 50  0001 C CNN
+F 2 "sictroller:Ceralink-L" H 3500 7150 50  0001 C CNN
 F 3 "" H 3500 7150 50  0000 C CNN
 	1    3500 7150
@@
 F 0 "C74" H 3710 7220 50  0000 L CNN
 F 1 "1uF" H 3710 7070 50  0000 L CNN
-F 2 "Capacitors_SMD:C_0603" H 3700 7150 50  0001 C CNN
+F 2 "sictroller:Ceralink-L" H 3700 7150 50  0001 C CNN
 F 3 "" H 3700 7150 50  0000 C CNN
 	1    3700 7150
@@
 F 0 "C75" H 3910 7220 50  0000 L CNN
 F 1 "1uF" H 3910 7070 50  0000 L CNN
-F 2 "Capacitors_SMD:C_0603" H 3900 7150 50  0001 C CNN
+F 2 "sictroller:Ceralink-L" H 3900 7150 50  0001 C CNN
 F 3 "" H 3900 7150 50  0000 C CNN
 	1    3900 7150
@@
 F 0 "C76" H 4110 7220 50  0000 L CNN
 F 1 "1uF" H 4110 7070 50  0000 L CNN
-F 2 "Capacitors_SMD:C_0603" H 4100 7150 50  0001 C CNN
+F 2 "sictroller:Ceralink-L" H 4100 7150 50  0001 C CNN
 F 3 "" H 4100 7150 50  0000 C CNN
 	1    4100 7150
@@
 F 0 "C77" H 4310 7220 50  0000 L CNN
 F 1 "1uF" H 4310 7070 50  0000 L CNN
-F 2 "Capacitors_SMD:C_0603" H 4300 7150 50  0001 C CNN
+F 2 "sictroller:Ceralink-L" H 4300 7150 50  0001 C CNN
 F 3 "" H 4300 7150 50  0000 C CNN
 	1    4300 7150
@@
 	4150 4250 4150 4650
 Wire Wire Line
-	3250 5550 3250 6300
-Connection ~ 3250 6050
-Connection ~ 3250 5950
-Wire Wire Line
-	3250 4250 3250 4750
+	3250 5550 3250 5750
+Wire Wire Line
+	3250 5850 3250 5950
 Connection ~ 3250 5850
-Connection ~ 3250 5650
 Wire Wire Line
 	1200 5450 3250 5450
@@
 	1200 4950 3250 4950
 Connection ~ 4150 4550
-Connection ~ 3250 4550
 Wire Wire Line
 	2950 4350 2950 4300
@@
 F 0 "J13" H 9850 6100 50  0000 C CNN
 F 1 "CONN_01X01" V 9950 6000 50  0000 C CNN
-F 2 "" H 9850 6000 50  0001 C CNN
+F 2 "Measurement_Points:Measurement_Point_Round-TH_Small" H 9850 6000 50  0001 C CNN
 F 3 "" H 9850 6000 50  0000 C CNN
 	1    9850 6000
@@
 Text Notes 8700 5650 0    60   ~ 0
 Y capacitor for heatsink
+Text Notes 3000 3750 0    60   ~ 0
+TODO: Softer level shifter?
+$Comp
+L TXS0108E U11
+U 1 1 5800B3B2
+P 3650 5350
+F 0 "U11" H 3450 4700 60  0000 L CNN
+F 1 "TXS0108E" H 3650 4700 60  0000 L CNN
+F 2 "sictroller:VQFN-20" H 3650 4650 60  0001 C CNN
+F 3 "" H 3650 4650 60  0000 C CNN
+	1    3650 5350
+	1    0    0    -1
+$EndComp
+Wire Wire Line
+	3250 4250 3250 4550
+$Comp
+L +3.3V #PWR0107
+U 1 1 5800C8BD
+P 3100 5650
+F 0 "#PWR0107" H 3100 5500 50  0001 C CNN
+F 1 "+3.3V" H 3100 5790 50  0000 C CNN
+F 2 "" H 3100 5650 50  0000 C CNN
+F 3 "" H 3100 5650 50  0000 C CNN
+	1    3100 5650
+	1    0    0    -1
+$EndComp
+Wire Wire Line
+	3100 5650 3250 5650
+Connection ~ 3250 5650
 $EndSCHEMATC

Commit message: Placement progress
Connections:
- net Y: now reaches C60.2, C61.1, J13.1 (P1), R54.2, R55.1
Changed lines of the file:
@@
 	3100 5650 3250 5650
 Connection ~ 3250 5650
+Text Label 9600 6000 0    60   ~ 0
+Y
 $EndSCHEMATC
