File: powerstage-CCS050M12CM2.sch (KiCad schematic (older format))
At the start: 46 parts, among them J13 CONN_01X01, Q2 CCS050M12CM2, U10 74LVC2G04, U11 TXS0108E

Commit message: Placement almost complete
Parts:
- removed R49, R50, R51, R52, R53, R55: 10k, Resistors_SMD:R_0402, symbol R_Small
Connections:
- net PWM_AH: now also U11.3 (A2); no longer U11.8 (A7)
- net PWM_AH_TTL: now also U11.18 (B2); no longer U11.13 (B7)
- net PWM_AL: now also U11.4 (A3); no longer R54.1, U11.7 (A6)
- net PWM_AL_TTL: now also U11.17 (B3); no longer U11.14 (B6)
- net PWM_BH: now also U11.5 (A4); no longer U11.6 (A5)
- net PWM_BH_TTL: now also U11.16 (B4); no longer U11.15 (B5)
- net PWM_BL: now also U11.6 (A5); no longer U11.5 (A4)
- net PWM_BL_TTL: now also U11.15 (B5); no longer U11.16 (B4)
- net PWM_CH: now also U11.7 (A6); no longer U11.4 (A3)
- net PWM_CH_TTL: now also U11.14 (B6); no longer U11.17 (B3)
- net PWM_CL: now also U11.8 (A7); no longer U11.3 (A2)
- net PWM_CL_TTL: now also U11.13 (B7); no longer U11.18 (B2)
- net ~PWR_RESET: now also R54.1
Other:
- note removed: "TODO: Softer level shifter?"
Changed lines of the file:
@@
-	1    0    0    -1
-$EndComp
-$Comp
-L R_Small R49
-U 1 1 57A190B9
-P 2600 4650
-F 0 "R49" H 2630 4670 50  0000 L CNN
-F 1 "10k" H 2630 4610 50  0000 L CNN
-F 2 "Resistors_SMD:R_0402" H 2600 4650 50  0001 C CNN
-F 3 "" H 2600 4650 50  0000 C CNN
-	1    2600 4650
 	1    0    0    -1
 $EndComp
@@
 $EndComp
 $Comp
-L +3.3V #PWR096
-U 1 1 57A19125
-P 2600 4500
-F 0 "#PWR096" H 2600 4350 50  0001 C CNN
-F 1 "+3.3V" H 2600 4640 50  0000 C CNN
-F 2 "" H 2600 4500 50  0000 C CNN
-F 3 "" H 2600 4500 50  0000 C CNN
-	1    2600 4500
-	1    0    0    -1
-$EndComp
-$Comp
-L GNDD #PWR097
+L GNDD #PWR096
 U 1 1 57A19193
 P 3250 5950
-F 0 "#PWR097" H 3250 5700 50  0001 C CNN
+F 0 "#PWR096" H 3250 5700 50  0001 C CNN
 F 1 "GNDD" H 3250 5800 50  0000 C CNN
 F 2 "" H 3250 5950 50  0000 C CNN
@@
 $EndComp
 $Comp
-L +3.3V #PWR098
+L +3.3V #PWR097
 U 1 1 57A19100
 P 3250 4250
-F 0 "#PWR098" H 3250 4100 50  0001 C CNN
+F 0 "#PWR097" H 3250 4100 50  0001 C CNN
 F 1 "+3.3V" H 3250 4390 50  0000 C CNN
 F 2 "" H 3250 4250 50  0000 C CNN
@@
 ~PWR_RESET
 Text HLabel 1200 5450 0    60   Input ~ 0
+PWM_CL
+Text HLabel 1200 5350 0    60   Input ~ 0
+PWM_CH
+Text HLabel 1200 5250 0    60   Input ~ 0
+PWM_BL
+Text HLabel 1200 5150 0    60   Input ~ 0
+PWM_BH
+Text HLabel 1200 5050 0    60   Input ~ 0
+PWM_AL
+Text HLabel 1200 4950 0    60   Input ~ 0
 PWM_AH
-Text HLabel 1200 5350 0    60   Input ~ 0
-PWM_AL
-Text HLabel 1200 5250 0    60   Input ~ 0
-PWM_BH
-Text HLabel 1200 5150 0    60   Input ~ 0
-PWM_BL
-Text HLabel 1200 5050 0    60   Input ~ 0
-PWM_CH
-Text HLabel 1200 4950 0    60   Input ~ 0
-PWM_CL
 Text Notes 3050 3950 0    60   ~ 0
 3.3V to 5V level conversion
@@
 $EndComp
 $Comp
-L GNDD #PWR099
+L GNDD #PWR098
 U 1 1 57A23C37
 P 2200 2150
-F 0 "#PWR099" H 2200 1900 50  0001 C CNN
+F 0 "#PWR098" H 2200 1900 50  0001 C CNN
 F 1 "GNDD" H 2200 2000 50  0000 C CNN
 F 2 "" H 2200 2150 50  0000 C CNN
@@
 $EndComp
 $Comp
-L +3.3V #PWR0100
+L +3.3V #PWR099
 U 1 1 57A23E25
 P 2200 1200
-F 0 "#PWR0100" H 2200 1050 50  0001 C CNN
+F 0 "#PWR099" H 2200 1050 50  0001 C CNN
 F 1 "+3.3V" H 2200 1340 50  0000 C CNN
 F 2 "" H 2200 1200 50  0000 C CNN
@@
 $EndComp
 $Comp
-L GNDD #PWR0101
+L GNDD #PWR0100
 U 1 1 57A244F4
 P 2500 1450
-F 0 "#PWR0101" H 2500 1200 50  0001 C CNN
+F 0 "#PWR0100" H 2500 1200 50  0001 C CNN
 F 1 "GNDD" H 2500 1300 50  0000 C CNN
 F 2 "" H 2500 1450 50  0000 C CNN
@@
 NoConn ~ 4150 5550
 Text Label 4850 5450 2    60   ~ 0
+PWM_CL_TTL
+Text Label 4850 5350 2    60   ~ 0
+PWM_CH_TTL
+Text Label 4850 5250 2    60   ~ 0
+PWM_BL_TTL
+Text Label 4850 5150 2    60   ~ 0
+PWM_BH_TTL
+Text Label 4850 5050 2    60   ~ 0
+PWM_AL_TTL
+Text Label 4850 4950 2    60   ~ 0
 PWM_AH_TTL
-Text Label 4850 5350 2    60   ~ 0
-PWM_AL_TTL
-Text Label 4850 5250 2    60   ~ 0
-PWM_BH_TTL
-Text Label 4850 5150 2    60   ~ 0
-PWM_BL_TTL
-Text Label 4850 5050 2    60   ~ 0
-PWM_CH_TTL
-Text Label 4850 4950 2    60   ~ 0
-PWM_CL_TTL
 Text Label 4850 4850 2    60   ~ 0
 ~PWR_RESET_TTL
@@
 GDRV_RDY_TTL
 $Comp
-L +5VD #PWR0102
+L +5VD #PWR0101
 U 1 1 57F46580
 P 5900 4750
-F 0 "#PWR0102" H 5900 4600 50  0001 C CNN
+F 0 "#PWR0101" H 5900 4600 50  0001 C CNN
 F 1 "+5VD" H 5900 4890 50  0000 C CNN
 F 2 "" H 5900 4750 50  0000 C CNN
@@
 $EndComp
 $Comp
-L GNDD #PWR0103
+L GNDD #PWR0102
 U 1 1 57F47836
 P 5900 5900
-F 0 "#PWR0103" H 5900 5650 50  0001 C CNN
+F 0 "#PWR0102" H 5900 5650 50  0001 C CNN
 F 1 "GNDD" H 5900 5750 50  0000 C CNN
 F 2 "" H 5900 5900 50  0000 C CNN
@@
 $EndComp
 $Comp
-L GNDD #PWR0104
+L GNDD #PWR0103
 U 1 1 57F48803
 P 5900 4000
-F 0 "#PWR0104" H 5900 3750 50  0001 C CNN
+F 0 "#PWR0103" H 5900 3750 50  0001 C CNN
 F 1 "GNDD" H 5900 3850 50  0000 C CNN
 F 2 "" H 5900 4000 50  0000 C CNN
@@
 $EndComp
 $Comp
-L GNDD #PWR0105
+L GNDD #PWR0104
 U 1 1 57F497CA
 P 5900 2100
-F 0 "#PWR0105" H 5900 1850 50  0001 C CNN
+F 0 "#PWR0104" H 5900 1850 50  0001 C CNN
 F 1 "GNDD" H 5900 1950 50  0000 C CNN
 F 2 "" H 5900 2100 50  0000 C CNN
@@
 $EndComp
 $Comp
-L +5VD #PWR0106
+L +5VD #PWR0105
 U 1 1 57F4B3DF
 P 5900 2850
-F 0 "#PWR0106" H 5900 2700 50  0001 C CNN
+F 0 "#PWR0105" H 5900 2700 50  0001 C CNN
 F 1 "+5VD" H 5900 2990 50  0000 C CNN
 F 2 "" H 5900 2850 50  0000 C CNN
@@
 $EndComp
 $Comp
-L +5VD #PWR0107
+L +5VD #PWR0106
 U 1 1 57F4C376
 P 5900 950
-F 0 "#PWR0107" H 5900 800 50  0001 C CNN
+F 0 "#PWR0106" H 5900 800 50  0001 C CNN
 F 1 "+5VD" H 5900 1090 50  0000 C CNN
 F 2 "" H 5900 950 50  0000 C CNN
@@
 BUS+
 $Comp
-L R_Small R50
-U 1 1 57F62930
-P 1400 5750
-F 0 "R50" H 1430 5770 50  0000 L CNN
-F 1 "10k" H 1430 5710 50  0000 L CNN
-F 2 "Resistors_SMD:R_0402" H 1400 5750 50  0001 C CNN
-F 3 "" H 1400 5750 50  0000 C CNN
-	1    1400 5750
-	1    0    0    -1
-$EndComp
-$Comp
-L R_Small R51
-U 1 1 57F62A97
-P 1700 5750
-F 0 "R51" H 1730 5770 50  0000 L CNN
-F 1 "10k" H 1730 5710 50  0000 L CNN
-F 2 "Resistors_SMD:R_0402" H 1700 5750 50  0001 C CNN
-F 3 "" H 1700 5750 50  0000 C CNN
-	1    1700 5750
-	1    0    0    -1
-$EndComp
-$Comp
-L R_Small R52
-U 1 1 57F62BEB
-P 2000 5750
-F 0 "R52" H 2030 5770 50  0000 L CNN
-F 1 "10k" H 2030 5710 50  0000 L CNN
-F 2 "Resistors_SMD:R_0402" H 2000 5750 50  0001 C CNN
-F 3 "" H 2000 5750 50  0000 C CNN
-	1    2000 5750
-	1    0    0    -1
-$EndComp
-$Comp
-L R_Small R53
-U 1 1 57F62E8A
-P 2300 5750
-F 0 "R53" H 2330 5770 50  0000 L CNN
-F 1 "10k" H 2330 5710 50  0000 L CNN
-F 2 "Resistors_SMD:R_0402" H 2300 5750 50  0001 C CNN
-F 3 "" H 2300 5750 50  0000 C CNN
-	1    2300 5750
-	1    0    0    -1
-$EndComp
-$Comp
 L R_Small R54
 U 1 1 57F62FB0
@@
 $EndComp
 $Comp
-L R_Small R55
-U 1 1 57F630D9
-P 2900 5750
-F 0 "R55" H 2930 5770 50  0000 L CNN
-F 1 "10k" H 2930 5710 50  0000 L CNN
-F 2 "Resistors_SMD:R_0402" H 2900 5750 50  0001 C CNN
-F 3 "" H 2900 5750 50  0000 C CNN
-	1    2900 5750
-	1    0    0    -1
-$EndComp
-$Comp
-L GNDD #PWR0108
-U 1 1 57F64D21
-P 1400 5950
-F 0 "#PWR0108" H 1400 5700 50  0001 C CNN
-F 1 "GNDD" H 1400 5800 50  0000 C CNN
-F 2 "" H 1400 5950 50  0000 C CNN
-F 3 "" H 1400 5950 50  0000 C CNN
-	1    1400 5950
-	1    0    0    -1
-$EndComp
-$Comp
-L GNDD #PWR0109
-U 1 1 57F6CC6B
-P 1700 5950
-F 0 "#PWR0109" H 1700 5700 50  0001 C CNN
-F 1 "GNDD" H 1700 5800 50  0000 C CNN
-F 2 "" H 1700 5950 50  0000 C CNN
-F 3 "" H 1700 5950 50  0000 C CNN
-	1    1700 5950
-	1    0    0    -1
-$EndComp
-$Comp
-L GNDD #PWR0110
-U 1 1 57F6CE7E
-P 2000 5950
-F 0 "#PWR0110" H 2000 5700 50  0001 C CNN
-F 1 "GNDD" H 2000 5800 50  0000 C CNN
-F 2 "" H 2000 5950 50  0000 C CNN
-F 3 "" H 2000 5950 50  0000 C CNN
-	1    2000 5950
-	1    0    0    -1
-$EndComp
-$Comp
-L GNDD #PWR0111
-U 1 1 57F6CE85
-P 2300 5950
-F 0 "#PWR0111" H 2300 5700 50  0001 C CNN
-F 1 "GNDD" H 2300 5800 50  0000 C CNN
-F 2 "" H 2300 5950 50  0000 C CNN
-F 3 "" H 2300 5950 50  0000 C CNN
-	1    2300 5950
-	1    0    0    -1
-$EndComp
-$Comp
-L GNDD #PWR0112
+L GNDD #PWR0107
 U 1 1 57F6D098
 P 2600 5950
-F 0 "#PWR0112" H 2600 5700 50  0001 C CNN
+F 0 "#PWR0107" H 2600 5700 50  0001 C CNN
 F 1 "GNDD" H 2600 5800 50  0000 C CNN
 F 2 "" H 2600 5950 50  0000 C CNN
 F 3 "" H 2600 5950 50  0000 C CNN
 	1    2600 5950
-	1    0    0    -1
-$EndComp
-$Comp
-L GNDD #PWR0113
-U 1 1 57F6D09F
-P 2900 5950
-F 0 "#PWR0113" H 2900 5700 50  0001 C CNN
-F 1 "GNDD" H 2900 5800 50  0000 C CNN
-F 2 "" H 2900 5950 50  0000 C CNN
-F 3 "" H 2900 5950 50  0000 C CNN
-	1    2900 5950
 	1    0    0    -1
 $EndComp
@@
 Text Notes 8700 5650 0    60   ~ 0
 Y capacitor for heatsink
-Text Notes 3000 3750 0    60   ~ 0
-TODO: Softer level shifter?
 $Comp
 L TXS0108E U11
@@
 $EndComp
 $Comp
-L +3.3V #PWR0114
+L +3.3V #PWR0108
 U 1 1 5800C8BD
 P 3100 5650
-F 0 "#PWR0114" H 3100 5500 50  0001 C CNN
+F 0 "#PWR0108" H 3100 5500 50  0001 C CNN
 F 1 "+3.3V" H 3100 5790 50  0000 C CNN
 F 2 "" H 3100 5650 50  0000 C CNN
@@
 Connection ~ 4150 4300
 Wire Wire Line
-	2600 4750 2600 4850
-Wire Wire Line
 	2500 4850 3250 4850
 Wire Wire Line
-	2600 4500 2600 4550
-Wire Wire Line
 	2200 2150 2200 2050
 Wire Wire Line
@@
 Wire Wire Line
 	2500 1200 2200 1200
-Connection ~ 2600 4850
 Wire Wire Line
 	4850 5450 4150 5450
@@
 	4150 4850 4850 4850
 Wire Wire Line
-	1200 5050 3250 5050
-Wire Wire Line
 	1200 5150 3250 5150
 Wire Wire Line
@@
 	5900 950  6150 950
 Wire Wire Line
-	1400 5950 1400 5850
-Wire Wire Line
-	2900 5650 2900 5450
-Connection ~ 2900 5450
-Wire Wire Line
-	2600 5650 2600 5350
-Connection ~ 2600 5350
-Wire Wire Line
-	2300 5650 2300 5250
-Connection ~ 2300 5250
-Wire Wire Line
-	2000 5650 2000 5150
-Connection ~ 2000 5150
-Wire Wire Line
-	1700 5650 1700 5050
-Connection ~ 1700 5050
-Wire Wire Line
-	1400 4950 1400 5650
-Connection ~ 1400 4950
-Wire Wire Line
-	1700 5950 1700 5850
-Wire Wire Line
-	2000 5950 2000 5850
-Wire Wire Line
-	2300 5950 2300 5850
+	2600 4850 2600 5650
 Wire Wire Line
 	2600 5950 2600 5850
-Wire Wire Line
-	2900 5950 2900 5850
 Connection ~ 4300 7250
 Connection ~ 4100 7250
@@
 Connection ~ 1900 7500
 Connection ~ 1900 7700
+Wire Wire Line
+	1200 5050 3250 5050
+Connection ~ 2600 4850
 $EndSCHEMATC

Commit message: Initial placement ~complete
Parts:
- added W2, W3: TEST_1P, Measurement_Points:Measurement_Point_Round-TH_Small, symbol TEST_1P
Connections:
- net PWM_AH_TTL: now also W2.1
- net PWM_AL_TTL: now also W3.1
Changed lines of the file:
@@
 	4850 5150 4150 5150
 Wire Wire Line
-	4850 5050 4150 5050
-Wire Wire Line
-	4850 4950 4150 4950
+	4150 5050 5150 5050
+Wire Wire Line
+	4150 4950 5000 4950
 Wire Wire Line
 	4150 4850 4850 4850
@@
 	1200 5050 3250 5050
 Connection ~ 2600 4850
+$Comp
+L TEST_1P W2
+U 1 1 58002D82
+P 5000 4950
+F 0 "W2" H 5000 5220 50  0000 C CNN
+F 1 "TEST_1P" H 5000 5150 50  0000 C CNN
+F 2 "Measurement_Points:Measurement_Point_Round-TH_Small" H 5200 4950 50  0001 C CNN
+F 3 "" H 5200 4950 50  0000 C CNN
+	1    5000 4950
+	1    0    0    -1
+$EndComp
+$Comp
+L TEST_1P W3
+U 1 1 580030CB
+P 5150 5050
+F 0 "W3" H 5150 5320 50  0000 C CNN
+F 1 "TEST_1P" H 5150 5250 50  0000 C CNN
+F 2 "Measurement_Points:Measurement_Point_Round-TH_Small" H 5350 5050 50  0001 C CNN
+F 3 "" H 5350 5050 50  0000 C CNN
+	1    5150 5050
+	1    0    0    -1
+$EndComp
 $EndSCHEMATC
