File: halfbridge-driver.sch (KiCad schematic (older format))
At the start: 29 parts, among them U1 MGJ1, U2 2ED020I12-F2, U3 MGJ1

Commit message: V2 schem complete, footprints not assigned
Parts:
- added C76, C78: 0.1u 50V, symbol C_Small
- added C82, C84: 0.1u 16V, symbol C_Small
- C75: renamed from C4; value 1u 35V -> 1u 50V
- C77: renamed from C7; value 1u 35V -> 1u 50V
- renumbered C1 to C79, C6 to C80, C5 to C81, C8 to C83, C2 to C85, C9 to C86, C3 to C87, C10 to C88, D6 to D10, D8 to D11, D4 to D12, D2 to D13, D5 to D6, D1 to D8, D3 to D9, R7 to R54, R1 to R55, R3 to R56, R5 to R57, R8 to R58, R4 to R59, R2 to R60, R6 to R61, U1 to U12, U3 to U13, U2 to U14
Connections:
- net +19V_HS: now also C76.1
- net +19V_LS: now also C78.1
- net -5V_HS: now also U12.3 (-V), U12.4 (-V), C82.2
- net -5V_LS: now also U13.3 (-V), U13.4 (-V), C84.2
- net SRC_H: now also C76.2, C82.1
- net SRC_L: now also C78.2, C84.1
- no-connect marks 0 -> 2
Other:
- moved on the sheet: C77, C80, C83, U13

Commit message: Add TVS protection to signal I/O.  Reannotate. Assign some footprints.
Parts:
- renumbered C75 to C78, C76 to C79, C77 to C80, C78 to C81, C79 to C82, C80 to C83, C81 to C84, C82 to C85, C83 to C86, C84 to C87, C85 to C88, C86 to C89, C87 to C90, C88 to C91, D7 to D10, D8 to D11, D9 to D12, D10 to D13, D11 to D14, D12 to D15, D13 to D16, D6 to D9, R54 to R56, R55 to R57, R56 to R58, R57 to R59, R58 to R60, R59 to R61, R60 to R62, R61 to R63

Commit message: Footprint assignment complete
Parts:
- C78, C80, C82, C83: footprint (none) -> Capacitors_SMD:C_0805
- C79, C81, C84, C86: footprint (none) -> Capacitors_SMD:C_0603
- C85, C87, C88, C89, C90, C91: footprint (none) -> Capacitors_SMD:C_0402
- D10, D11, D12, D14, D15, D16: footprint (none) -> Diodes_SMD:SOD-523
- D13, D9: footprint (none) -> Diodes_SMD:SMA_Standard
- R56, R57, R59, R60, R62, R63: footprint (none) -> Resistors_SMD:R_0402
- R58, R61: footprint (none) -> sictroller:MELF-0204
- U12, U13: footprint (none) -> sictroller:MGJ1
- U14: footprint (none) -> sictroller:PG-DSO-36-58

Commit message: Placement progress
Connections:
- net DESAT_LS: now reaches C91.1, D15.1 (K), R60.2, U14.20 (DESATLS)
- net DRVL: now reaches R61.2, U14.23 (OUTLS)
- net DESAT_HS: now reaches C89.1, D12.1 (K), R56.2, U14.30 (DESATHS)
- net DRVH: now reaches R58.2, U14.34 (OUTHS)
Changed lines of the file:
@@
 $Descr A4 11693 8268
 encoding utf-8
-Sheet 6 8
+Sheet 7 8
 Title ""
 Date ""
@@
 	4000 1400 4000 1500
 Connection ~ 4000 1450
+Text Label 6650 3150 0    60   ~ 0
+DESAT_HS
+Text Label 6650 4350 0    60   ~ 0
+DESAT_LS
+Text Label 6100 3350 0    60   ~ 0
+DRVH
+Text Label 6100 4550 0    60   ~ 0
+DRVL
 $EndSCHEMATC

Commit message: Power stage / gate drive approx placement complete
Parts:
- R59, R63: footprint Resistors_SMD:R_0402 -> Resistors_SMD:R_0805
Changed lines of the file:
@@
 AR Path="/57A1662D/57F2705F/57F02200" Ref="U20"  Part="1"
 AR Path="/57F02200" Ref="U14"  Part="1"
-F 0 "U14" H 4450 2750 60  0000 L BNN
+F 0 "U20" H 4450 2750 60  0000 L BNN
 F 1 "2ED020I12-F2" H 5950 2750 60  0000 R BNN
 F 2 "sictroller:PG-DSO-36-58" H 5200 4050 60  0001 C CNN
@@
 AR Path="/57A1662D/57F260F4/57F05C45" Ref="U15"  Part="1"
 AR Path="/57A1662D/57F2705F/57F05C45" Ref="U18"  Part="1"
-F 0 "U12" H 3350 900 40  0000 L BNN
+F 0 "U18" H 3350 900 40  0000 L BNN
 F 1 "MGJ1" H 3900 900 30  0000 R BNN
 F 2 "sictroller:MGJ1" H 3550 1250 60  0001 C CNN
@@
 AR Path="/57A1662D/57F260F4/57F05D03" Ref="C96"  Part="1"
 AR Path="/57A1662D/57F2705F/57F05D03" Ref="C110"  Part="1"
-F 0 "C82" H 3110 1320 50  0000 L CNN
+F 0 "C110" H 3110 1320 50  0000 L CNN
 F 1 "10u 16V" H 3110 1170 50  0000 L CNN
 F 2 "Capacitors_SMD:C_0805" H 3100 1250 50  0001 C CNN
@@
 AR Path="/57A1662D/57F260F4/57F05DBD" Ref="C92"  Part="1"
 AR Path="/57A1662D/57F2705F/57F05DBD" Ref="C106"  Part="1"
-F 0 "C78" H 4460 1220 50  0000 L CNN
+F 0 "C106" H 4460 1220 50  0000 L CNN
 F 1 "1u 50V" H 4460 1070 50  0000 L CNN
 F 2 "Capacitors_SMD:C_0805" H 4450 1150 50  0001 C CNN
@@
 AR Path="/57A1662D/57F260F4/57F05E19" Ref="C98"  Part="1"
 AR Path="/57A1662D/57F2705F/57F05E19" Ref="C112"  Part="1"
-F 0 "C84" H 4460 1420 50  0000 L CNN
+F 0 "C112" H 4460 1420 50  0000 L CNN
 F 1 "1u 16V" H 4460 1270 50  0000 L CNN
 F 2 "Capacitors_SMD:C_0603" H 4450 1350 50  0001 C CNN
@@
 AR Path="/57A1662D/57F260F4/57F0708D" Ref="U16"  Part="1"
 AR Path="/57A1662D/57F2705F/57F0708D" Ref="U19"  Part="1"
-F 0 "U13" H 7550 900 40  0000 L BNN
+F 0 "U19" H 7550 900 40  0000 L BNN
 F 1 "MGJ1" H 8100 900 30  0000 R BNN
 F 2 "sictroller:MGJ1" H 7750 1250 60  0001 C CNN
@@
 AR Path="/57A1662D/57F260F4/57F07093" Ref="C97"  Part="1"
 AR Path="/57A1662D/57F2705F/57F07093" Ref="C111"  Part="1"
-F 0 "C83" H 7310 1320 50  0000 L CNN
+F 0 "C111" H 7310 1320 50  0000 L CNN
 F 1 "10u 16V" H 7310 1170 50  0000 L CNN
 F 2 "Capacitors_SMD:C_0805" H 7300 1250 50  0001 C CNN
@@
 AR Path="/57A1662D/57F260F4/57F07099" Ref="C94"  Part="1"
 AR Path="/57A1662D/57F2705F/57F07099" Ref="C108"  Part="1"
-F 0 "C80" H 8660 1220 50  0000 L CNN
+F 0 "C108" H 8660 1220 50  0000 L CNN
 F 1 "1u 50V" H 8660 1070 50  0000 L CNN
 F 2 "Capacitors_SMD:C_0805" H 8650 1150 50  0001 C CNN
@@
 AR Path="/57A1662D/57F260F4/57F0709F" Ref="C100"  Part="1"
 AR Path="/57A1662D/57F2705F/57F0709F" Ref="C114"  Part="1"
-F 0 "C86" H 8660 1420 50  0000 L CNN
+F 0 "C114" H 8660 1420 50  0000 L CNN
 F 1 "1u 16V" H 8660 1270 50  0000 L CNN
 F 2 "Capacitors_SMD:C_0603" H 8650 1350 50  0001 C CNN
@@
 AR Path="/57A1662D/57F260F4/57F1574E" Ref="R66"  Part="1"
 AR Path="/57A1662D/57F2705F/57F1574E" Ref="R74"  Part="1"
-F 0 "R58" V 6350 3200 50  0000 L CNN
+F 0 "R74" V 6350 3200 50  0000 L CNN
 F 1 "10R MELF" V 6550 3200 50  0000 L CNN
 F 2 "sictroller:MELF-0204" H 6450 3350 50  0001 C CNN
@@
 AR Path="/57A1662D/57F260F4/57F16BC4" Ref="D17"  Part="1"
 AR Path="/57A1662D/57F2705F/57F16BC4" Ref="D25"  Part="1"
-F 0 "D9" H 8650 3230 50  0000 L CNN
+F 0 "D25" H 8650 3230 50  0000 L CNN
 F 1 "HV" H 8550 3070 50  0000 L CNN
 F 2 "Diodes_SMD:SMA_Standard" V 8700 3150 50  0001 C CNN
@@
 AR Path="/57A1662D/57F260F4/57F16C61" Ref="D18"  Part="1"
 AR Path="/57A1662D/57F2705F/57F16C61" Ref="D26"  Part="1"
-F 0 "D10" H 9050 3250 50  0000 C CNN
+F 0 "D26" H 9050 3250 50  0000 C CNN
 F 1 "4.3V" H 9050 3050 50  0000 C CNN
 F 2 "Diodes_SMD:SOD-523" H 9050 3150 50  0001 C CNN
@@
 AR Path="/57A1662D/57F260F4/57F16FB9" Ref="R64"  Part="1"
 AR Path="/57A1662D/57F2705F/57F16FB9" Ref="R72"  Part="1"
-F 0 "R56" V 8250 3000 50  0000 L CNN
+F 0 "R72" V 8250 3000 50  0000 L CNN
 F 1 "1k" V 8450 3000 50  0000 L CNN
 F 2 "Resistors_SMD:R_0402" H 8350 3150 50  0001 C CNN
@@
 AR Path="/57A1662D/57F260F4/57F17070" Ref="C103"  Part="1"
 AR Path="/57A1662D/57F2705F/57F17070" Ref="C117"  Part="1"
-F 0 "C89" H 8060 3520 50  0000 L CNN
+F 0 "C117" H 8060 3520 50  0000 L CNN
 F 1 "220pF" H 8060 3370 50  0000 L CNN
 F 2 "Capacitors_SMD:C_0402" H 8050 3450 50  0001 C CNN
@@
 AR Path="/57A1662D/57F260F4/57F185FE" Ref="R67"  Part="1"
 AR Path="/57A1662D/57F2705F/57F185FE" Ref="R75"  Part="1"
-F 0 "R59" H 6600 3500 50  0000 L CNN
+F 0 "R75" H 6600 3500 50  0000 L CNN
 F 1 "47k" H 6550 3600 50  0000 L CNN
-F 2 "Resistors_SMD:R_0402" H 6750 3550 50  0001 C CNN
+F 2 "Resistors_SMD:R_0805" H 6750 3550 50  0001 C CNN
 F 3 "" H 6750 3550 50  0000 C CNN
 	1    6750 3550
@@
 AR Path="/57A1662D/57F260F4/57F1899B" Ref="D20"  Part="1"
 AR Path="/57A1662D/57F2705F/57F1899B" Ref="D28"  Part="1"
-F 0 "D12" V 7500 3600 50  0000 C CNN
+F 0 "D28" V 7500 3600 50  0000 C CNN
 F 1 "10V" V 7700 3650 50  0000 C CNN
 F 2 "Diodes_SMD:SOD-523" H 7650 3500 50  0001 C CNN
@@
 AR Path="/57A1662D/57F260F4/57F19BF8" Ref="R69"  Part="1"
 AR Path="/57A1662D/57F2705F/57F19BF8" Ref="R77"  Part="1"
-F 0 "R61" V 6350 4400 50  0000 L CNN
+F 0 "R77" V 6350 4400 50  0000 L CNN
 F 1 "10R MELF" V 6550 4400 50  0000 L CNN
 F 2 "sictroller:MELF-0204" H 6450 4550 50  0001 C CNN
@@
 AR Path="/57A1662D/57F260F4/57F19C08" Ref="D21"  Part="1"
 AR Path="/57A1662D/57F2705F/57F19C08" Ref="D29"  Part="1"
-F 0 "D13" H 8650 4430 50  0000 L CNN
+F 0 "D29" H 8650 4430 50  0000 L CNN
 F 1 "HV" H 8550 4270 50  0000 L CNN
 F 2 "Diodes_SMD:SMA_Standard" V 8700 4350 50  0001 C CNN
@@
 AR Path="/57A1662D/57F260F4/57F19C0E" Ref="D22"  Part="1"
 AR Path="/57A1662D/57F2705F/57F19C0E" Ref="D30"  Part="1"
-F 0 "D14" H 9050 4450 50  0000 C CNN
+F 0 "D30" H 9050 4450 50  0000 C CNN
 F 1 "4.3V" H 9050 4250 50  0000 C CNN
 F 2 "Diodes_SMD:SOD-523" H 9050 4350 50  0001 C CNN
@@
 AR Path="/57A1662D/57F260F4/57F19C16" Ref="R68"  Part="1"
 AR Path="/57A1662D/57F2705F/57F19C16" Ref="R76"  Part="1"
-F 0 "R60" V 8250 4200 50  0000 L CNN
+F 0 "R76" V 8250 4200 50  0000 L CNN
 F 1 "1k" V 8450 4200 50  0000 L CNN
 F 2 "Resistors_SMD:R_0402" H 8350 4350 50  0001 C CNN
@@
 AR Path="/57A1662D/57F260F4/57F19C1F" Ref="C105"  Part="1"
 AR Path="/57A1662D/57F2705F/57F19C1F" Ref="C119"  Part="1"
-F 0 "C91" H 8060 4720 50  0000 L CNN
+F 0 "C119" H 8060 4720 50  0000 L CNN
 F 1 "220pF" H 8060 4570 50  0000 L CNN
 F 2 "Capacitors_SMD:C_0402" H 8050 4650 50  0001 C CNN
@@
 AR Path="/57A1662D/57F260F4/57F19C2A" Ref="R71"  Part="1"
 AR Path="/57A1662D/57F2705F/57F19C2A" Ref="R79"  Part="1"
-F 0 "R63" H 6600 4700 50  0000 L CNN
+F 0 "R79" H 6600 4700 50  0000 L CNN
 F 1 "47k" H 6550 4800 50  0000 L CNN
-F 2 "Resistors_SMD:R_0402" H 6750 4750 50  0001 C CNN
+F 2 "Resistors_SMD:R_0805" H 6750 4750 50  0001 C CNN
 F 3 "" H 6750 4750 50  0000 C CNN
 	1    6750 4750
@@
 AR Path="/57A1662D/57F260F4/57F19C34" Ref="D23"  Part="1"
 AR Path="/57A1662D/57F2705F/57F19C34" Ref="D31"  Part="1"
-F 0 "D15" V 7500 4800 50  0000 C CNN
+F 0 "D31" V 7500 4800 50  0000 C CNN
 F 1 "10V" V 7700 4850 50  0000 C CNN
 F 2 "Diodes_SMD:SOD-523" H 7650 4700 50  0001 C CNN
@@
 AR Path="/57A1662D/57F260F4/57F1A51C" Ref="C102"  Part="1"
 AR Path="/57A1662D/57F2705F/57F1A51C" Ref="C116"  Part="1"
-F 0 "C88" H 3410 3170 50  0000 L CNN
+F 0 "C116" H 3410 3170 50  0000 L CNN
 F 1 "0.1u 16V" H 3410 3020 50  0000 L CNN
 F 2 "Capacitors_SMD:C_0402" H 3400 3100 50  0001 C CNN
@@
 AR Path="/57A1662D/57F260F4/57F1C1CA" Ref="R65"  Part="1"
 AR Path="/57A1662D/57F2705F/57F1C1CA" Ref="R73"  Part="1"
-F 0 "R57" V 2650 3200 50  0000 L CNN
+F 0 "R73" V 2650 3200 50  0000 L CNN
 F 1 "1k" V 2850 3200 50  0000 L CNN
 F 2 "Resistors_SMD:R_0402" H 2750 3350 50  0001 C CNN
@@
 AR Path="/57A1662D/57F260F4/57F1C51E" Ref="D19"  Part="1"
 AR Path="/57A1662D/57F2705F/57F1C51E" Ref="D27"  Part="1"
-F 0 "D11" V 3050 3300 50  0000 L CNN
+F 0 "D27" V 3050 3300 50  0000 L CNN
 F 1 "D_Schottky_Small" V 2950 2700 50  0000 L CNN
 F 2 "Diodes_SMD:SOD-523" V 3000 3450 50  0001 C CNN
@@
 AR Path="/57A1662D/57F260F4/57F1DED1" Ref="C104"  Part="1"
 AR Path="/57A1662D/57F2705F/57F1DED1" Ref="C118"  Part="1"
-F 0 "C90" H 3410 4470 50  0000 L CNN
+F 0 "C118" H 3410 4470 50  0000 L CNN
 F 1 "0.1u 16V" H 3410 4320 50  0000 L CNN
 F 2 "Capacitors_SMD:C_0402" H 3400 4400 50  0001 C CNN
@@
 AR Path="/57A1662D/57F260F4/57F1DEE0" Ref="R70"  Part="1"
 AR Path="/57A1662D/57F2705F/57F1DEE0" Ref="R78"  Part="1"
-F 0 "R62" V 2650 4500 50  0000 L CNN
+F 0 "R78" V 2650 4500 50  0000 L CNN
 F 1 "1k" V 2850 4500 50  0000 L CNN
 F 2 "Resistors_SMD:R_0402" H 2750 4650 50  0001 C CNN
@@
 AR Path="/57A1662D/57F260F4/57F1DEE7" Ref="D24"  Part="1"
 AR Path="/57A1662D/57F2705F/57F1DEE7" Ref="D32"  Part="1"
-F 0 "D16" V 3050 4600 50  0000 L CNN
+F 0 "D32" V 3050 4600 50  0000 L CNN
 F 1 "D_Schottky_Small" V 2950 4000 50  0000 L CNN
 F 2 "Diodes_SMD:SOD-523" V 3000 4750 50  0001 C CNN
@@
 AR Path="/57A1662D/57F260F4/57FC6B04" Ref="C95"  Part="1"
 AR Path="/57A1662D/57F2705F/57FC6B04" Ref="C109"  Part="1"
-F 0 "C81" H 9010 1220 50  0000 L CNN
+F 0 "C109" H 9010 1220 50  0000 L CNN
 F 1 "0.1u 50V" H 9010 1070 50  0000 L CNN
 F 2 "Capacitors_SMD:C_0603" H 9000 1150 50  0001 C CNN
@@
 AR Path="/57A1662D/57F260F4/57FC6BF3" Ref="C101"  Part="1"
 AR Path="/57A1662D/57F2705F/57FC6BF3" Ref="C115"  Part="1"
-F 0 "C87" H 9010 1420 50  0000 L CNN
+F 0 "C115" H 9010 1420 50  0000 L CNN
 F 1 "0.1u 16V" H 9010 1270 50  0000 L CNN
 F 2 "Capacitors_SMD:C_0402" H 9000 1350 50  0001 C CNN
@@
 AR Path="/57A1662D/57F260F4/57FC72B1" Ref="C93"  Part="1"
 AR Path="/57A1662D/57F2705F/57FC72B1" Ref="C107"  Part="1"
-F 0 "C79" H 4810 1220 50  0000 L CNN
+F 0 "C107" H 4810 1220 50  0000 L CNN
 F 1 "0.1u 50V" H 4810 1070 50  0000 L CNN
 F 2 "Capacitors_SMD:C_0603" H 4800 1150 50  0001 C CNN
@@
 AR Path="/57A1662D/57F260F4/57FC72B7" Ref="C99"  Part="1"
 AR Path="/57A1662D/57F2705F/57FC72B7" Ref="C113"  Part="1"
-F 0 "C85" H 4810 1420 50  0000 L CNN
+F 0 "C113" H 4810 1420 50  0000 L CNN
 F 1 "0.1u 16V" H 4810 1270 50  0000 L CNN
 F 2 "Capacitors_SMD:C_0402" H 4800 1350 50  0001 C CNN
