File: halfbridge-driver.sch (KiCad schematic (older format))
At the start: 33 parts, among them U12 MGJ1, U13 MGJ1, U14 2ED020I12-F2

Commit message: Add more ceralinks on rear
Parts:
- renumbered C87 to C100, C88 to C101, C89 to C102, C90 to C103, C91 to C104, C78 to C91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
