File: sictroller.kicad_pcb (KiCad board)
At the start: 6 copper layers, 135.8 x 121.3 mm, 323 parts, among them J1 CONN_01X02, J10 CONN_01X02, J11 RINGTERM, J12 RINGTERM, J14 CONN_01X05, J15 CONN_01X03, J2 CONN_01X08, J3 CONN_02X05, J4 RINGTERM, J5 RINGTERM, J6 RINGTERM, J7 CONN_01X02, J8 RINGTERM, J9 RINGTERM, Q1 CSD17483F4, Q2 CCS050M12CM2, T1 7508110151, U1 ACPL-M61L, U10 74LVC2G04, U11 TXS0108E, U12 MGJ1, U13 MGJ1, U14 2ED020I12-F2, U15 MGJ1, U16 MGJ1, U17 2ED020I12-F2, U18 MGJ1, U19 MGJ1, U2 TMS320F28069M, U20 2ED020I12-F2, U3 ADM3053, U4 TPS76201, U5 TPS76201, U6 XCL221B18, U7 VIPER26HD, U8 ADUM5241, U9 MAX6691, Y1 CSTCE20M0V13C

Commit message: Silkscreen done both sides, added aux LED
Parts:
- added D34: LED, LEDs:LED_0603, F.Cu at (117.8, 132.7)
- added R51: 330, Resistors_SMD:R_0402, B.Cu at (117.8, 131.4)
Routing:
- net Net-(D34-Pad1): track 0.00 -> 2.37 mm
- net +3V3: track 98.6 -> 100.7 mm
- net Net-(D34-Pad2): track 0.00 -> 1.46 mm, vias 0 -> 1
Other:
- board text added: "| | | / \ ___| * |___ | /\ | || || || || """ """"
